File: projects/PCB schematics/USER/USER.sch (EAGLE design)
At the start: 84 parts, among them IC1 OP11D, IC10 74AHC1G32DCK, IC13 OP11D, IC14 74AHC1G32DCK, IC17 OP11D, IC18 74AHC1G32DCK, IC19 OP11D, IC20 OP11D, IC3 OP11D, IC4 OP11D, IC5 OP11D, IC6 74AHC1G32DCK, IC7 OP11D, IC8 OP11D, IC9 74AHC1G32DCK

Commit message: SC - Rev A; First PCB revision complete.
This marks the first draft of the SC board.
Parts have been laid out and initial routing completed through
extensive use of autorouter.
Other:
- note removed: "1. Preconditioning - APPS1"
- note removed: "1. Preconditioning - APPS2"
- note removed: "1. Preconditioning - BOTS"
- note removed: "1. Preconditioning - HVD"
- note removed: "1. Preconditioning - INERTIA"
- note removed: "2. Plausibility - APPS1"
- note removed: "2. Plausibility - APPS2"
- note removed: "2. Plausibility - BOTS"
- note removed: "2. Plausibility - HVD"
- note removed: "2. Plausibility - INERTIA"
- note removed: "Plausibility Sensitivity Threshold"
- note removed: "Voltage References"
- moved on the sheet: C10, C11, C6, C7, IC10, IC6, R17, R18, R3, R4
