File: projects/PCB schematics/CSC/CSC.brd (EAGLE design)
At the start: 160 x 100 mm, 23 parts, among them Q1 IRLZ44Z, Q2 IRLZ44Z

Commit message: TSMPC - Initial draft (WIP).
Non-working commit of TSMPC.
Done simply to show possible board layout.
Parts:
- moved Q2 347.8 mm to (88.9, 78.7)
- moved R5 314.1 mm to (45.7, 68.6)
- moved BUF3 287.6 mm to (127.0, 26.7)
- moved C2 285.2 mm to (45.7, 53.3)
- moved R4 285.2 mm to (45.7, 58.4)
- moved SDB-CHARGE 247.2 mm to (106.7, 92.7)
- moved INT1 247.2 mm to (106.7, 69.8)
- moved INT2 247.2 mm to (106.7, 81.3)
- moved AIR- 167.8 mm to (19.1, 83.8)
- moved D2 160.1 mm to (12.7, 61.0)
- moved BUF2 145.1 mm to (127.0, 41.9)
- moved S1 140.6 mm to (139.7, 10.2)
- moved BUF1 129.6 mm to (127.0, 55.9)
- moved C1 116.1 mm to (57.1, 52.1)
- moved R1 116.1 mm to (62.2, 52.1)
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