File: projects/PCB schematics/BSPD/BSPD.sch (EAGLE design)
At the start: 60 parts, among them IC1 LM741D, IC10 74AHC1G32DCK, IC2 LM741D, IC3 OP11D, IC4 OP11D, IC5 OP11D, IC6 OP11D, IC7 74AHC1G32DCK, IC9 NE555D

Commit message: SC - Rev A; First PCB revision complete.
This marks the first draft of the SC board.
Parts have been laid out and initial routing completed through
extensive use of autorouter.
Other:
- note removed: "1. BSE signal acq. & conditioning"
- note removed: "1. Motor current signal acq. & conditioning"
- note removed: "2. Fault condition"
- note removed: "3. 100 Hz Clock"
- note removed: "3. Fault Signal Persistence Counter"
- note removed: "4. No-Fault Counter Reset"
- note removed: "BSE Plausibility Check"
- note removed: "Implausibility Sensitivity"
- note removed: "Motor Current Signal Plausibility Check"
- note removed: "Voltage references"
- moved on the sheet: AND1A, AND1B, AND1C, AND2A, AND2B, AND3A, C8, C9, NOT1, OR1A, OR1B, OR2A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

Commit message: SC - Rev C; SC70 -> SOT23.
For single logic gate components, SC70 was initially chosen.
These packages proved too small to hand-solder.

All SC70 packages have been refactored to SOT23.

SparkFun DRC's added in for additional manufacturability.
Parts:
- IC10, IC7, OR3: value 74AHC1G32DCK -> 74AHC1G32DBV; device 74xx-little-de:74AHC1G32DCK -> 74xx-little-de:74AHC1G32DBV
- NOT1: value 74AHC1G04DCK -> 74AHC1G04DBV; device 74xx-little-us:74AHC1G04DCK -> 74xx-little-us:74AHC1G04DBV
- R7: value 15k -> (none)
Connections:
- new net N$61: IC9.DIS, R33.1, R7.2
- net N$22: no longer R7.1
- net THR: now also R7.1; no longer R33.1, R7.2
Other:
- moved on the sheet: C8, R33

Commit message: BSPD - Schematic revision/component revision.
During ESF, schematics chosen used European part libraries.
These were updated to US symbols, with appropriate final parts sourced
to allow builds of both SOP8 and DIL-8 packages.
Parts:
- removed AND1: 74ALS09D, 74xx-eu:74ALS09D
- removed AND2, AND3: 74HC13D, 74xx-eu:74HC13D
- removed NOT1: 74AHC1G04DBV, 74xx-little-us:74AHC1G04DBV
- removed OR1, OR2: 4072D, 40xx:4072D
- removed OR3: 74AHC1G32DBV, 74xx-little-de:74AHC1G32DBV
- removed R19: 12k, rcl:R-US_R0805
- removed R32: 1k, rcl:R-US_R0805
- removed R33: (no value), rcl:R-US_R0805
- removed RESETCOUNT, SIGNALCOUNT: 4020D, 40xx:4020D
- added C10, C11, C12, C13, C14, C15: 0.01uF, rcl:C-EUC0805
- added IC11: 4020D, 40xx:4020D
- added IC12, IC13: 74LS32D, 74xx-us:74LS32D
- added IC8: 74ALS09D, 74xx-us:74ALS09D
- added JP1, JP2, JP3, JP4, JP5, JP6, JP7, JP8: (no value), con-lstb:MA03-1
- added RN1, RN2, RN4: (no value), resistor-dil:15RSOMC
- added SV1, SV2, SV3, SV4, SV5, SV6: (no value), con-lstb:MA07-2
- added X1: 5566-2, con-molex:5566-2
- C1: device rcl:C-EUC0805 -> rcl:CPOL-US085CS-1AR
- C5: device rcl:CPOL-US085CS-1AR -> rcl:C-EUC0805
- C8: value 10uF -> 0.01uF; device rcl:CPOL-US085CS-1AW -> rcl:C-EUC0805
- C9: value 0.01uF -> 470nF
- IC1, IC2: value LM741D -> OP11D; device linear:LM741D -> linear:OP11D
- IC10, IC7: value 74AHC1G32DBV -> 74LS32D; device 74xx-little-de:74AHC1G32DBV -> 74xx-us:74LS32D
- IC3: value OP11D -> 74LS32D; device linear:OP11D -> 74xx-us:74LS32D; SPICEPREFIX (none) -> J
- IC4: value OP11D -> NE555D; device linear:OP11D -> linear:NE555D
- IC5: value OP11D -> 4020D; device linear:OP11D -> 40xx:4020D
- IC9: value NE555D -> 74AHC1G04DBV; device linear:NE555D -> 74xx-little-us:74AHC1G04DBV
- R1: value (none) -> 50k
- R11, R12, R5: value 10k -> 50k
- R16: value (none) -> 470; device rcl:R-TRIMM3224X -> rcl:R-US_R0805
- R17: value (none) -> 470
- R18, R2, R7: value (none) -> 10k
- R20, R22: value 27k -> 10k
- R21: value 12k -> 10k
- R23, R24, R25, R26, R27, R28, R29, R30, R31: value 1k -> 10k
- R3, R4: value (none) -> 10k; device rcl:R-TRIMM3224X -> rcl:R-US_R0805
Connections:
- removed net BSE: R19.2
- removed net BSE_P: IC1.+IN, IC3A.+IN, IC3B.-IN, IC4A.OUT
- removed net BSPDFAULT: OR3A.O
- removed net MOTCUR: R21.2
- removed net MOTCUR_P: IC2.+IN, IC5A.+IN, IC5B.-IN, IC6A.OUT
- removed net N$18: IC6A.-IN, R28.1, R29.1
- removed net THR: C8.+, IC9.THR, IC9.TR, R7.1
- new net BSE_PROCESSED: IC2A.+IN, IC2B.-IN, IC6A.+IN
- new net MOTCUR_PROCESSED: IC1A.+IN, IC1B.-IN, IC6B.+IN
- new net N$62: RN4.7, SV1.3
- new net N$63: RN4.8, SV1.1
- new net N$64: RN4.15, SV2.14
- new net N$65: RN4.14, SV2.12
- new net N$66: RN4.13, SV2.10
- new net N$67: RN4.12, SV2.8
- new net N$68: RN4.11, SV2.6
- new net N$69: RN4.10, SV2.4
- new net N$70: IC5A.Q11, JP8.1
- new net N$71: RN1.2, SV3.13
- new net N$72: RN1.3, SV3.11
- new net N$73: RN1.4, SV3.9
- new net N$74: RN1.5, SV3.7
- new net N$75: RN1.6, SV3.5
- new net N$76: RN1.7, SV3.3
- new net N$77: RN1.8, SV3.1
- new net N$78: RN1.15, SV4.14
- new net N$79: RN1.14, SV4.12
- new net N$80: RN1.13, SV4.10
- new net N$81: RN1.12, SV4.8
- new net N$82: RN1.11, SV4.6
- new net N$83: RN1.10, SV4.4
- new net N$84: RN2.2, SV5.13
- new net N$85: RN2.3, SV5.11
- new net N$86: RN2.4, SV5.9
- new net N$87: RN2.5, SV5.7
- new net N$88: RN2.6, SV5.5
- new net N$89: RN2.7, SV5.3
- new net N$90: RN2.8, SV5.1
- new net N$91: RN2.15, SV6.14
- new net N$92: RN2.14, SV6.12
- new net N$93: RN2.13, SV6.10
- new net N$94: RN2.12, SV6.8
- new net N$95: RN2.11, SV6.6
- new net N$96: RN2.10, SV6.4
- new net N$97: IC5A.Q9, JP2.1
- new net N$98: R18.2
- new net N$99: JP1.3, JP2.3, JP3.3, JP7.3, JP8.3
- new net TR: C9.1, IC4.THR, IC4.TR, R17.1
- net +0.5V: now also IC1B.+IN, IC2B.+IN, R14.2, R9.1; no longer IC3B.+IN, IC5B.+IN, R14.1, R15.2
- net +1.0V: now also R4.1, R9.2; no longer R13.1, R14.2, R24.2, R29.2
- net +4.0V: now also R13.2, R8.1; no longer R6.1, R8.2
- net +4.5V: now also IC1A.-IN, IC2A.-IN, R2.1, R8.2; no longer IC3A.-IN, IC5A.-IN, R5.1, R6.2
- net +5V: now also C1.+, C2.1, IC4.R, IC4.V+, R16.2, R2.2, RN1.1, RN2.1, RN4.1, SV1.10, SV1.12, SV1.14, SV1.2, SV1.4, SV1.6, SV1.8, SV3.10, SV3.12, SV3.14, SV3.2, SV3.4, SV3.6, SV3.8, SV5.10, SV5.12, SV5.14, SV5.2, SV5.4, SV5.6, SV5.8, X1-1.S; no longer AND3A.I3, C4.1, C5.+, IC9.R, IC9.V+, R16.E, R3.E, R33.2, R4.E, R5.2
- net BSPDPLAUS1: now also IC3A.O; no longer IC7A.O
- net BSPDPLAUS2: now also IC3B.O; no longer IC10A.O
- net GND: now also C1.-, C10.2, C11.2, C12.2, C13.2, C14.2, C15.2, C5.2, C8.1, C9.2, IC4.GND, JP4.3, JP5.3, JP6.3, R14.1, R18.1, R21.1, R23.1, R24.1, R25.1, R26.1, R27.1, R28.1, R29.1, R30.1, R31.1, R6.1, RN1.9, RN2.9, RN4.9, SV2.1, SV2.11, SV2.13, SV2.2, SV2.3, SV2.5, SV2.7, SV2.9, SV4.1, SV4.11, SV4.13, SV4.2, SV4.3, SV4.5, SV4.7, SV4.9, SV6.1, SV6.11, SV6.13, SV6.2, SV6.3, SV6.5, SV6.7, SV6.9, X1-2.S; no longer C1.2, C5.-, C8.-, C9.1, IC9.GND, OR2A.I3, R15.1, R16.A, R25.2, R27.2, R3.A, R30.2, R32.2, R4.A
- net N$1: now also R13.1, R15.2; no longer IC3A.OUT, R1.1
- net N$10: now also C7.1, IC2D.+IN, R12.2; no longer C2.1, IC3C.+IN, R1.2
- net N$11: now also IC1A.OUT, R1.1; no longer C1.1, IC3D.+IN, R2.2
- net N$12: now also C4.1, IC1C.+IN, R1.2; no longer C6.1, IC5C.+IN, R17.2
- net N$13: now also C6.1, IC1D.+IN, R11.2; no longer C7.1, IC5D.+IN, R18.2
- net N$14: now also IC1B.OUT, R11.1; no longer IC5B.OUT, R18.1
- net N$15: now also IC3C.I1; no longer IC6A.+IN, R30.1, R31.2
- net N$16: now also RN4.2, SV1.13; no longer R21.1, R22.2, R28.2
- net N$17: now also IC13C.O, IC3D.I1; no longer R31.1, R32.1
- net N$19: now also C10.1, C11.1, IC6A.-IN, RN4.16; no longer IC1.-IN, R3.S
- net N$2: now also R10.2, R15.1; no longer R8.1, R9.2
- net N$20: now also IC7C.I0, JP1.2; no longer R19.1, R23.2
- net N$21: now also C12.1, C13.1, IC6B.-IN, RN1.16; no longer IC2.-IN, R4.S
- net N$22: now also IC4.Q, IC8B.I0, IC8C.I1; no longer AND1B.I0, AND1C.I1, IC9.Q
- net N$23: now also IC13B.O, IC3D.I0; no longer R26.1, R27.1
- net N$24: now also IC10C.I0, JP4.2, R21.2; no longer IC4A.-IN, R23.1, R24.1
- net N$25: now also C8.2, IC4.CV; no longer C9.2, IC9.CV
- net N$26: now also IC6B.OUT, IC8A.I1; no longer AND1A.I1, IC2.OUT
- net N$27: now also IC6A.OUT, IC8A.I0; no longer AND1A.I0, IC1.OUT
- net N$28: now also IC11A.RES, IC8A.O, IC8B.I1, IC9A.I; no longer AND1A.O, AND1B.I1, NOT1A.I, RESETCOUNTA.RES
- net N$29: now also IC8C.I0, IC9A.O; no longer AND1C.I0, NOT1A.O
- net N$3: now also IC3C.I0, IC5A.Q14, R6.2; no longer IC4A.+IN, R25.1, R26.2
- net N$30: now also IC11A.P1, IC8C.O; no longer AND1C.O, RESETCOUNTA.P1
- net N$31: now also IC11A.Q10, JP5.1; no longer OR1A.I0, RESETCOUNTA.Q6
- net N$32: now also IC11A.Q9, JP4.1; no longer OR1A.I1, RESETCOUNTA.Q7
- net N$33: now also IC10C.I1, JP5.2, R22.2; no longer OR1A.I2, RESETCOUNTA.Q8
- net N$34: now also IC10C.O, IC12B.I0; no longer OR1A.I3, RESETCOUNTA.Q9
- net N$35: now also IC10D.O, IC12B.I1; no longer OR1B.I0, RESETCOUNTA.Q10
- net N$36: now also IC12A.O, IC12C.I1; no longer OR1B.I1, RESETCOUNTA.Q11
- net N$37: now also IC10D.I0, JP6.2, R23.2; no longer OR1B.I2, RESETCOUNTA.Q12
- net N$38: now also IC11A.Q11, JP6.1; no longer OR1B.I3, RESETCOUNTA.Q13
- net N$39: now also IC12B.O, IC12C.I0; no longer OR1A.O, OR2A.I0
- net N$4: now also R3.2, R7.1; no longer R10.2, R9.1
- net N$40: now also IC5A.Q8, JP1.1; no longer OR1B.O, OR2A.I1
- net N$41: now also IC7C.I1, JP2.2, R27.2; no longer OR2A.I2, RESETCOUNTA.Q14
- net N$42: now also IC12C.O, IC5A.RES; no longer OR2A.O, SIGNALCOUNTA.RES
- net N$43: now also IC5A.P1, IC8B.O; no longer AND1B.O, SIGNALCOUNTA.P1
- net N$44: now also IC2C.OUT, IC3A.I0; no longer IC3C.OUT, IC7A.I0
- net N$45: now also IC2D.OUT, IC3A.I1; no longer IC3D.OUT, IC7A.I1
- net N$46: now also IC1C.OUT, IC3B.I0; no longer IC10A.I0, IC5C.OUT
- net N$47: now also IC1D.OUT, IC3B.I1; no longer IC10A.I1, IC5D.OUT
- net N$48: now also IC7D.I0, JP3.2, R28.2; no longer AND2A.O, AND3A.I0
- net N$49: now also IC5A.Q10, JP3.1; no longer AND2B.O, AND3A.I1
- net N$5: now also R3.1, R4.2; no longer R11.1, R12.2
- net N$50: now also IC7D.I1, JP8.2, R29.2; no longer AND2B.I3, SIGNALCOUNTA.Q12
- net N$51: now also IC13A.I0, IC5A.Q12, R30.2; no longer AND2B.I2, SIGNALCOUNTA.Q11
- net N$52: now also IC10D.I1, IC11A.Q12, R24.2; no longer AND2B.I1, SIGNALCOUNTA.Q10
- net N$53: now also IC11A.Q13, IC12A.I0, R25.2; no longer AND2B.I0, SIGNALCOUNTA.Q9
- net N$54: now also IC11A.Q14, IC12A.I1, R26.2; no longer AND2A.I3, SIGNALCOUNTA.Q8
- net N$55: now also IC13A.I1, IC5A.Q13, R31.2; no longer AND2A.I2, SIGNALCOUNTA.Q7
- net N$56: now also IC7D.O; no longer AND2A.I1, SIGNALCOUNTA.Q6
- net N$57: now also RN4.3, SV1.11; no longer AND2A.I0, SIGNALCOUNTA.Q5
- net N$58: now also RN4.4, SV1.9; no longer AND3A.I2, SIGNALCOUNTA.Q13
- net N$59: now also RN4.5, SV1.7; no longer OR3A.I1, SIGNALCOUNTA.Q14
- net N$6: now also R10.1, R7.2; no longer IC5A.OUT, R17.1
- net N$60: now also RN4.6, SV1.5; no longer AND3A.O, OR3A.I0
- net N$61: now also IC4.DIS, R16.1, R17.2; no longer IC9.DIS, R33.1, R7.2
- net N$7: now also IC2A.OUT, R5.1; no longer R12.1, R13.2
- net N$8: now also IC2B.OUT, R12.1; no longer IC3B.OUT, R2.1
- net N$9: now also C5.1, IC2C.+IN, R5.2; no longer R10.1, R11.2
- net TIME_THRESH: now also C14.1, C15.1, IC1C.-IN, IC1D.-IN, IC2C.-IN, IC2D.-IN, RN2.16; no longer IC3C.-IN, IC3D.-IN, IC5C.-IN, IC5D.-IN, R16.S
Other:
- note added: "03/24/19"
- note added: "1. BSPDFAULT 2. BSPDPLAUS1 3. BSPDPLAUS2 4. IMDFAULT 5. BMSFAULT 6. TEMPFAULT 7. FUSEFAULT 8. AUX1 9. AUX2 10. SCU control signal 11. Reset main fault"
- note added: "1. BSPDLED 2. BSPDPLAUS1LED 3. BSPDPLAUS2LED 4. IMDLED 5. BMSLED 6. TEMPLED 7. FUSELED 8. AUX1LED 9. AUX2LED 10. AIR Control"
- note added: "1. VCC (+5V) 2. GND"
- note added: "Author: github.com/michaelpass"
- note added: "C = 470nF, R1 = 470, R2 = 470 1021Hz, 66.67% duty cycle"
- note added: "Inputs:"
- note added: "Outputs:"
- note added: "Power:"
- note added: "Short/open-circuit detection"
- note removed: "11/30/18"
- note removed: "Author: Michael Pass"
- moved on the sheet: C2, C3, C4, C6, C7, C9, IC6A, R1, R10, R11, R12, R13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

Commit message: TSALC - Initial build.
Initial build done by Anshuman. 
TSALC is still WIP.
TSALC work must be continued on another branch.
Changed lines of the file:
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@@
 <wire x1="35.56" y1="228.6" x2="27.94" y2="228.6" width="0.1524" layer="91"/>
 <junction x="35.56" y="228.6"/>
-<wire x1="35.56" y1="233.68" x2="35.56" y2="228.6" width="0.1524" layer="91"/>
 <pinref part="P+1" gate="1" pin="+5V"/>
 <wire x1="35.56" y1="228.6" x2="35.56" y2="231.14" width="0.1524" layer="91"/>
@@
 <label x="393.7" y="190.5" size="1.778" layer="95" rot="R180" xref="yes"/>
 <wire x1="393.7" y1="190.5" x2="406.4" y2="190.5" width="0.1524" layer="91"/>
+<junction x="406.4" y="190.5"/>
 </segment>
 </net>
@@
 <junction x="355.6" y="129.54"/>
 <pinref part="C9" gate="G$1" pin="1"/>
+<junction x="340.36" y="129.54"/>
 </segment>
 </net>
@@
 <wire x1="436.88" y1="-22.86" x2="439.42" y2="-22.86" width="0.1524" layer="91"/>
 <pinref part="IC8" gate="C" pin="O"/>
+<junction x="439.42" y="-22.86"/>
 </segment>
 </net>
@@
 <wire x1="142.24" y1="205.74" x2="147.32" y2="205.74" width="0.1524" layer="91"/>
 <label x="147.32" y="205.74" size="1.778" layer="95" xref="yes"/>
+<junction x="142.24" y="205.74"/>
 </segment>
 <segment>
@@
 <wire x1="175.26" y1="193.04" x2="180.34" y2="193.04" width="0.1524" layer="91"/>
 <label x="180.34" y="193.04" size="1.778" layer="95" xref="yes"/>
+<junction x="175.26" y="193.04"/>
 </segment>
 <segment>
@@
 <wire x1="581.66" y1="210.82" x2="581.66" y2="208.28" width="0.1524" layer="91"/>
 <junction x="581.66" y="210.82"/>
+<junction x="457.2" y="226.06"/>
 </segment>
 </net>
@@
 <wire x1="584.2" y1="-22.86" x2="581.66" y2="-22.86" width="0.1524" layer="91"/>
 <wire x1="571.5" y1="-22.86" x2="584.2" y2="-22.86" width="0.1524" layer="91"/>
+<junction x="584.2" y="-22.86"/>
 </segment>
 </net>
@@
 </sheet>
 </sheets>
+<errors>
+</errors>
 </schematic>
 </drawing>

Commit message: BSPD - Schematic finalized.
BSPD schematic needed final refactoring for parts.
Adjustable threshold settings have been put in for plausibility checks
using resistor arrays.

Squashed - BSPD - Removed BSPD.brd.

Too much work will be required to refactor this board.
It's currently 10 inches long.
Given the work entailed, I'm scrapping the board and relaying from a clean slate.

Squashed - BSPD - Created BSPD.brd.

Board file created.
Parts:
- removed IC13: 74LS32D, 74xx-us:74LS32D
- added JP10, JP9: (no value), con-lstb:MA03-1
- added R19: 10k, rcl:R-US_R0805
- added R32, R33, R34: 50k, rcl:R-US_R0805
- added X2: 5566-2, con-molex:5566-2
- added X3: 5566-4, con-molex:5566-4
- IC10: value 74LS32D -> 4020D; device 74xx-us:74LS32D -> 40xx:4020D
- IC11: value 4020D -> 74LS32D; device 40xx:4020D -> 74xx-us:74LS32D
- R26: value 10k -> 50k
Connections:
- removed net N$24: IC10C.I0, JP4.2, R21.2
- removed net N$28: IC11A.RES, IC8A.O, IC8B.I1, IC9A.I
- removed net N$30: IC11A.P1, IC8C.O
- new net BSPDFAULT: IC7D.O, X3-3.S
- new net N$100: IC5A.Q12, JP7.1
- new net N$101: IC10A.Q12, JP10.1
- new net N$102: IC11C.O, IC11D.I1
- new net N$103: IC11A.O, IC12A.I0
- new net N$104: IC11B.O, IC12A.I1
- new net N$105: IC11D.O, IC12B.I1
- new net N$18: IC3C.O, IC7C.I0
- new net RESET_FAULTCOUNT: IC12B.O, IC5A.RES
- net +5V: now also R26.2, R33.2
- net BSE_PROCESSED: now also R26.1, R32.2, X2-1.S
- net BSPDPLAUS1: now also X3-1.S
- net BSPDPLAUS2: now also X3-2.S
- net GND: now also R19.1, R32.1, R34.1; no longer JP4.3, JP5.3, JP6.3, R26.1
- net MOTCUR_PROCESSED: now also R33.1, R34.2, X2-2.S
- net N$15: now also IC7A.O, IC7B.I1; no longer IC3C.I1
- net N$17: now also IC10A.RES, IC8A.O, IC8B.I1, IC9A.I; no longer IC13C.O, IC3D.I1
- net N$20: now also IC3C.I0; no longer IC7C.I0
- net N$23: now also IC7C.O, IC7D.I0; no longer IC13B.O, IC3D.I0
- net N$3: now also IC7B.I0; no longer IC3C.I0
- net N$31: now also IC11A.I0, JP4.2, R18.2; no longer IC11A.Q10, JP5.1
- net N$32: now also IC10A.Q8; no longer IC11A.Q9
- net N$33: now also IC11A.I1, R19.2; no longer IC10C.I1, R22.2
- net N$34: now also IC11B.I0, JP6.2, R21.2; no longer IC10C.O, IC12B.I0
- net N$35: now also IC10A.Q10, JP6.1; no longer IC10D.O, IC12B.I1
- net N$36: now also IC11B.I1, JP9.2, R22.2; no longer IC12A.O, IC12C.I1
- net N$37: now also IC11C.I0, JP10.2; no longer IC10D.I0, JP6.2
- net N$38: now also IC10A.Q13, IC11C.I1, R24.2; no longer IC11A.Q11, JP6.1
- net N$39: now also IC10A.Q9, JP5.1; no longer IC12B.O, IC12C.I0
- net N$41: now also IC3C.I1; no longer IC7C.I1
- net N$42: now also IC10A.P1, IC8C.O; no longer IC12C.O, IC5A.RES
- net N$48: now also IC3D.I0; no longer IC7D.I0
- net N$50: now also IC3D.I1; no longer IC7D.I1
- net N$51: now also IC7A.I0, JP7.2; no longer IC13A.I0, IC5A.Q12
- net N$52: now also IC10A.Q11, JP9.1; no longer IC10D.I1, IC11A.Q12, R24.2
- net N$53: now also IC12A.O, IC12B.I0; no longer IC11A.Q13, IC12A.I0, R25.2
- net N$54: now also IC10A.Q14, IC11D.I0, R25.2; no longer IC11A.Q14, IC12A.I1, R26.2
- net N$55: now also IC7A.I1; no longer IC13A.I1
- net N$56: now also IC3D.O, IC7C.I1; no longer IC7D.O
- net N$98: now also IC7B.O, IC7D.I1; no longer R18.2
- net N$99: now also JP10.3, JP4.3, JP5.3, JP6.3, JP9.3
Other:
- note added: "1. BSE_PROCESSED 2. MOTCUR_PROCESSED"
- note added: "1. BSPDPLAUS1 2. BSPDPLAUS2 3. BSPDFAULT"
- note added: "C = 470nF, R1 = 470, R2 = 470 2173Hz, 66.67% duty cycle"
- note removed: "1. BSPDFAULT 2. BSPDPLAUS1 3. BSPDPLAUS2 4. IMDFAULT 5. BMSFAULT 6. TEMPFAULT 7. FUSEFAULT 8. AUX1 9. AUX2 10. SCU control signal 11. Reset main fault"
- note removed: "1. BSPDLED 2. BSPDPLAUS1LED 3. BSPDPLAUS2LED 4. IMDLED 5. BMSLED 6. TEMPLED 7. FUSELED 8. AUX1LED 9. AUX2LED 10. AIR Control"
- note removed: "C = 470nF, R1 = 470, R2 = 470 1021Hz, 66.67% duty cycle"
- moved on the sheet: C1, C10, C11, C12, C13, C14, C15, C2, C3, C4, C5, C6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

Commit message: BSPD - Initial placement.
Parts have been laid down in a preliminary placement. Routing for power will first be done, and then autorouting will be caried out for signals. Autorouting must be reviewed and redone manually.
Parts:
- removed RN4: (no value), resistor-dil:15RSOMC
- added RN3: (no value), resistor-dil:15RSOMC
- C1: device rcl:CPOL-US085CS-1AR -> rcl:C-EUC0805
- renumbered IC1 to OP2, IC10 to COUNT2, IC11 to OR3, IC12 to OR4, IC2 to OP1, IC3 to OR1, IC4 to NE555D, IC5 to COUNT1, IC6 to OP3, IC7 to OR2, IC8 to AND1, IC9 to NOT1
Connections:
- net +5V: now also C1.1, RN3.1; no longer C1.+, RN4.1
- net GND: now also C1.2, RN3.9; no longer C1.-, RN4.9
- net N$100: now also JP5.1; no longer JP7.1
- net N$16: now also RN1.2; no longer RN4.2
- net N$19: now also RN1.16; no longer RN4.16
- net N$21: now also RN2.16; no longer RN1.16
- net N$31: now also JP6.2; no longer JP4.2
- net N$32: now also JP6.1; no longer JP4.1
- net N$33: now also JP7.2; no longer JP5.2
- net N$34: now also JP8.2; no longer JP6.2
- net N$35: now also JP8.1; no longer JP6.1
- net N$39: now also JP7.1; no longer JP5.1
- net N$50: now also JP4.2; no longer JP8.2
- net N$51: now also JP5.2; no longer JP7.2
- net N$57: now also RN1.3; no longer RN4.3
- net N$58: now also RN1.4; no longer RN4.4
- net N$59: now also RN1.5; no longer RN4.5
- net N$60: now also RN1.6; no longer RN4.6
- net N$62: now also RN1.7; no longer RN4.7
- net N$63: now also RN1.8; no longer RN4.8
- net N$64: now also RN1.15; no longer RN4.15
- net N$65: now also RN1.14; no longer RN4.14
- net N$66: now also RN1.13; no longer RN4.13
- net N$67: now also RN1.12; no longer RN4.12
- net N$68: now also RN1.11; no longer RN4.11
- net N$69: now also RN1.10; no longer RN4.10
- net N$70: now also JP4.1; no longer JP8.1
- net N$71: now also RN2.2; no longer RN1.2
- net N$72: now also RN2.3; no longer RN1.3
- net N$73: now also RN2.4; no longer RN1.4
- net N$74: now also RN2.5; no longer RN1.5
- net N$75: now also RN2.6; no longer RN1.6
- net N$76: now also RN2.7; no longer RN1.7
- net N$77: now also RN2.8; no longer RN1.8
- net N$78: now also RN2.15; no longer RN1.15
- net N$79: now also RN2.14; no longer RN1.14
- net N$80: now also RN2.13; no longer RN1.13
- net N$81: now also RN2.12; no longer RN1.12
- net N$82: now also RN2.11; no longer RN1.11
- net N$83: now also RN2.10; no longer RN1.10
- net N$84: now also RN3.2; no longer RN2.2
- net N$85: now also RN3.3; no longer RN2.3
- net N$86: now also RN3.4; no longer RN2.4
- net N$87: now also RN3.5; no longer RN2.5
- net N$88: now also RN3.6; no longer RN2.6
- net N$89: now also RN3.7; no longer RN2.7
- net N$90: now also RN3.8; no longer RN2.8
- net N$91: now also RN3.15; no longer RN2.15
- net N$92: now also RN3.14; no longer RN2.14
- net N$93: now also RN3.13; no longer RN2.13
- net N$94: now also RN3.12; no longer RN2.12
- net N$95: now also RN3.11; no longer RN2.11
- net N$96: now also RN3.10; no longer RN2.10
- net TIME_THRESH: now also RN3.16; no longer RN2.16
Other:
- moved on the sheet: JP4, JP5, JP6, JP7, JP8, RN1, RN2

Commit message: BSPD - Hand routing complete.
Proceding with auto routing.

Squashed - BSPD - Initial routing.

Routing underway. Ground pour chosen. Routing easy choices before attempting autorouting.
Connections:
- net +5V: now also AND1P.VCC, COUNT1P.VDD, COUNT2P.VDD, NOT1P.VCC, OP1P.V+, OP2P.V+, OP3P.V+, OR1P.VCC, OR2P.VCC, OR3P.VCC, OR4P.VCC
- net GND: now also AND1P.GND, COUNT1P.VSS, COUNT2P.VSS, NOT1P.GND, OP1P.V-, OP2P.V-, OP3P.V-, OR1P.GND, OR2P.GND, OR3P.GND, OR4P.GND
