File: projects/PCB schematics/BSPD/BSPD.sch (EAGLE design)
At the start: 83 parts, among them X1 5566-2, X2 5566-2, X3 5566-4

Commit message: BSPD - Rev A; Gerber files.
Initial board revisions complete. This board represents a working draft. GERBER files have been generated. Please review.
Connections:
- removed net N$99: JP1.3, JP10.3, JP2.3, JP3.3, JP4.3, JP5.3, JP6.3, JP7.3, JP8.3, JP9.3
- net GND: now also JP1.3, JP10.3, JP2.3, JP3.3, JP4.3, JP5.3, JP6.3, JP7.3, JP8.3, JP9.3
Changed lines of the file:
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@@
 <wire x1="283.972" y1="144.78" x2="283.972" y2="141.732" width="0.1524" layer="91"/>
+</segment>
+<segment>
+<pinref part="JP6" gate="G$1" pin="3"/>
+<wire x1="426.72" y1="129.54" x2="426.72" y2="132.08" width="0.1524" layer="91"/>
+<wire x1="426.72" y1="132.08" x2="436.88" y2="132.08" width="0.1524" layer="91"/>
+<wire x1="436.88" y1="60.96" x2="436.88" y2="132.08" width="0.1524" layer="91"/>
+<pinref part="JP7" gate="G$1" pin="3"/>
+<wire x1="426.72" y1="111.76" x2="426.72" y2="114.3" width="0.1524" layer="91"/>
+<wire x1="426.72" y1="114.3" x2="439.42" y2="114.3" width="0.1524" layer="91"/>
+<wire x1="439.42" y1="60.96" x2="439.42" y2="114.3" width="0.1524" layer="91"/>
+<pinref part="JP8" gate="G$1" pin="3"/>
+<wire x1="426.72" y1="93.98" x2="426.72" y2="96.52" width="0.1524" layer="91"/>
+<wire x1="426.72" y1="96.52" x2="441.96" y2="96.52" width="0.1524" layer="91"/>
+<wire x1="441.96" y1="96.52" x2="441.96" y2="60.96" width="0.1524" layer="91"/>
+<pinref part="GND18" gate="1" pin="GND"/>
+<wire x1="447.04" y1="76.2" x2="447.04" y2="60.96" width="0.1524" layer="91"/>
+<pinref part="JP9" gate="G$1" pin="3"/>
+<wire x1="447.04" y1="60.96" x2="447.04" y2="55.88" width="0.1524" layer="91"/>
+<pinref part="JP10" gate="G$1" pin="3"/>
+<wire x1="426.72" y1="76.2" x2="447.04" y2="76.2" width="0.1524" layer="91"/>
+<wire x1="426.72" y1="58.42" x2="426.72" y2="60.96" width="0.1524" layer="91"/>
+<wire x1="426.72" y1="60.96" x2="436.88" y2="60.96" width="0.1524" layer="91"/>
+<junction x="447.04" y="60.96"/>
+<wire x1="436.88" y1="60.96" x2="439.42" y2="60.96" width="0.1524" layer="91"/>
+<wire x1="439.42" y1="60.96" x2="441.96" y2="60.96" width="0.1524" layer="91"/>
+<wire x1="441.96" y1="60.96" x2="447.04" y2="60.96" width="0.1524" layer="91"/>
+<junction x="441.96" y="60.96"/>
+<junction x="439.42" y="60.96"/>
+<junction x="436.88" y="60.96"/>
+</segment>
+<segment>
+<pinref part="JP1" gate="G$1" pin="3"/>
+<wire x1="426.72" y1="266.7" x2="426.72" y2="269.24" width="0.1524" layer="91"/>
+<wire x1="426.72" y1="269.24" x2="436.88" y2="269.24" width="0.1524" layer="91"/>
+<wire x1="436.88" y1="198.12" x2="436.88" y2="269.24" width="0.1524" layer="91"/>
+<pinref part="JP2" gate="G$1" pin="3"/>
+<wire x1="426.72" y1="248.92" x2="426.72" y2="251.46" width="0.1524" layer="91"/>
+<wire x1="426.72" y1="251.46" x2="439.42" y2="251.46" width="0.1524" layer="91"/>
+<wire x1="439.42" y1="198.12" x2="439.42" y2="251.46" width="0.1524" layer="91"/>
+<pinref part="JP3" gate="G$1" pin="3"/>
+<wire x1="426.72" y1="231.14" x2="426.72" y2="233.68" width="0.1524" layer="91"/>
+<wire x1="426.72" y1="233.68" x2="441.96" y2="233.68" width="0.1524" layer="91"/>
+<wire x1="441.96" y1="233.68" x2="441.96" y2="198.12" width="0.1524" layer="91"/>
+<pinref part="GND13" gate="1" pin="GND"/>
+<wire x1="447.04" y1="213.36" x2="447.04" y2="198.12" width="0.1524" layer="91"/>
+<pinref part="JP4" gate="G$1" pin="3"/>
+<wire x1="447.04" y1="198.12" x2="447.04" y2="193.04" width="0.1524" layer="91"/>
+<pinref part="JP5" gate="G$1" pin="3"/>
+<wire x1="426.72" y1="213.36" x2="447.04" y2="213.36" width="0.1524" layer="91"/>
+<wire x1="426.72" y1="195.58" x2="426.72" y2="198.12" width="0.1524" layer="91"/>
+<wire x1="426.72" y1="198.12" x2="436.88" y2="198.12" width="0.1524" layer="91"/>
+<junction x="447.04" y="198.12"/>
+<wire x1="436.88" y1="198.12" x2="439.42" y2="198.12" width="0.1524" layer="91"/>
+<wire x1="439.42" y1="198.12" x2="441.96" y2="198.12" width="0.1524" layer="91"/>
+<wire x1="441.96" y1="198.12" x2="447.04" y2="198.12" width="0.1524" layer="91"/>
+<junction x="441.96" y="198.12"/>
+<junction x="439.42" y="198.12"/>
+<junction x="436.88" y="198.12"/>
 </segment>
 </net>
@@
 </segment>
 </net>
-<net name="N$99" class="0">
-<segment>
-<pinref part="JP1" gate="G$1" pin="3"/>
-<wire x1="426.72" y1="266.7" x2="426.72" y2="269.24" width="0.1524" layer="91"/>
-<wire x1="426.72" y1="269.24" x2="436.88" y2="269.24" width="0.1524" layer="91"/>
-<wire x1="436.88" y1="198.12" x2="436.88" y2="269.24" width="0.1524" layer="91"/>
-<pinref part="JP2" gate="G$1" pin="3"/>
-<wire x1="426.72" y1="248.92" x2="426.72" y2="251.46" width="0.1524" layer="91"/>
-<wire x1="426.72" y1="251.46" x2="439.42" y2="251.46" width="0.1524" layer="91"/>
-<wire x1="439.42" y1="198.12" x2="439.42" y2="251.46" width="0.1524" layer="91"/>
-<pinref part="JP3" gate="G$1" pin="3"/>
-<wire x1="426.72" y1="231.14" x2="426.72" y2="233.68" width="0.1524" layer="91"/>
-<wire x1="426.72" y1="233.68" x2="441.96" y2="233.68" width="0.1524" layer="91"/>
-<wire x1="441.96" y1="233.68" x2="441.96" y2="198.12" width="0.1524" layer="91"/>
-<pinref part="GND13" gate="1" pin="GND"/>
-<wire x1="447.04" y1="213.36" x2="447.04" y2="198.12" width="0.1524" layer="91"/>
-<pinref part="JP4" gate="G$1" pin="3"/>
-<wire x1="447.04" y1="198.12" x2="447.04" y2="193.04" width="0.1524" layer="91"/>
-<pinref part="JP5" gate="G$1" pin="3"/>
-<wire x1="426.72" y1="213.36" x2="447.04" y2="213.36" width="0.1524" layer="91"/>
-<wire x1="426.72" y1="195.58" x2="426.72" y2="198.12" width="0.1524" layer="91"/>
-<wire x1="426.72" y1="198.12" x2="436.88" y2="198.12" width="0.1524" layer="91"/>
-<junction x="447.04" y="198.12"/>
-<wire x1="436.88" y1="198.12" x2="439.42" y2="198.12" width="0.1524" layer="91"/>
-<wire x1="439.42" y1="198.12" x2="441.96" y2="198.12" width="0.1524" layer="91"/>
-<wire x1="441.96" y1="198.12" x2="447.04" y2="198.12" width="0.1524" layer="91"/>
-<junction x="441.96" y="198.12"/>
-<junction x="439.42" y="198.12"/>
-<junction x="436.88" y="198.12"/>
-</segment>
-<segment>
-<pinref part="JP6" gate="G$1" pin="3"/>
-<wire x1="426.72" y1="129.54" x2="426.72" y2="132.08" width="0.1524" layer="91"/>
-<wire x1="426.72" y1="132.08" x2="436.88" y2="132.08" width="0.1524" layer="91"/>
-<wire x1="436.88" y1="60.96" x2="436.88" y2="132.08" width="0.1524" layer="91"/>
-<pinref part="JP7" gate="G$1" pin="3"/>
-<wire x1="426.72" y1="111.76" x2="426.72" y2="114.3" width="0.1524" layer="91"/>
-<wire x1="426.72" y1="114.3" x2="439.42" y2="114.3" width="0.1524" layer="91"/>
-<wire x1="439.42" y1="60.96" x2="439.42" y2="114.3" width="0.1524" layer="91"/>
-<pinref part="JP8" gate="G$1" pin="3"/>
-<wire x1="426.72" y1="93.98" x2="426.72" y2="96.52" width="0.1524" layer="91"/>
-<wire x1="426.72" y1="96.52" x2="441.96" y2="96.52" width="0.1524" layer="91"/>
-<wire x1="441.96" y1="96.52" x2="441.96" y2="60.96" width="0.1524" layer="91"/>
-<pinref part="GND18" gate="1" pin="GND"/>
-<wire x1="447.04" y1="76.2" x2="447.04" y2="60.96" width="0.1524" layer="91"/>
-<pinref part="JP9" gate="G$1" pin="3"/>
-<wire x1="447.04" y1="60.96" x2="447.04" y2="55.88" width="0.1524" layer="91"/>
-<pinref part="JP10" gate="G$1" pin="3"/>
-<wire x1="426.72" y1="76.2" x2="447.04" y2="76.2" width="0.1524" layer="91"/>
-<wire x1="426.72" y1="58.42" x2="426.72" y2="60.96" width="0.1524" layer="91"/>
-<wire x1="426.72" y1="60.96" x2="436.88" y2="60.96" width="0.1524" layer="91"/>
-<junction x="447.04" y="60.96"/>
-<wire x1="436.88" y1="60.96" x2="439.42" y2="60.96" width="0.1524" layer="91"/>
-<wire x1="439.42" y1="60.96" x2="441.96" y2="60.96" width="0.1524" layer="91"/>
-<wire x1="441.96" y1="60.96" x2="447.04" y2="60.96" width="0.1524" layer="91"/>
-<junction x="441.96" y="60.96"/>
-<junction x="439.42" y="60.96"/>
-<junction x="436.88" y="60.96"/>
-</segment>
-</net>
