File: projects/PCB schematics/POWER/POWER-DCDC.brd (EAGLE design)
At the start: 160 x 100 mm, 1 part

Commit message: RTDS - Rev A.
Other:
- board size 160 x 100 mm -> 99.1 x 99.1 mm
Changed lines of the file:
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@@
 <?xml version="1.0" encoding="utf-8"?>
 <!DOCTYPE eagle SYSTEM "eagle.dtd">
-<eagle version="9.3.2">
+<eagle version="9.4.0">
 <drawing>
 <settings>
@@
 <board>
 <plain>
-<wire x1="0" y1="0" x2="160" y2="0" width="0" layer="20"/>
-<wire x1="160" y1="0" x2="160" y2="100" width="0" layer="20"/>
-<wire x1="160" y1="100" x2="0" y2="100" width="0" layer="20"/>
-<wire x1="0" y1="100" x2="0" y2="0" width="0" layer="20"/>
+<wire x1="0" y1="0" x2="99.06" y2="0" width="0" layer="20"/>
+<wire x1="99.06" y1="0" x2="99.06" y2="99.06" width="0" layer="20"/>
+<wire x1="99.06" y1="99.06" x2="0" y2="99.06" width="0" layer="20"/>
+<wire x1="0" y1="99.06" x2="0" y2="0" width="0" layer="20"/>
 </plain>
 <attributes>
@@
 </class>
 </classes>
-<designrules name="default">
-<description language="de">&lt;b&gt;EAGLE Design Rules&lt;/b&gt;
-&lt;p&gt;
-Die Standard-Design-Rules sind so gewählt, dass sie für
-die meisten Anwendungen passen. Sollte ihre Platine
-besondere Anforderungen haben, treffen Sie die erforderlichen
-Einstellungen hier und speichern die Design Rules unter
-einem neuen Namen ab.</description>
+<designrules name="default *">
 <description language="en">&lt;b&gt;EAGLE Design Rules&lt;/b&gt;
 &lt;p&gt;
@@
 <param name="mtCopper" value="0.035mm 0.035mm 0.035mm 0.035mm 0.035mm 0.035mm 0.035mm 0.035mm 0.035mm 0.035mm 0.035mm 0.035mm 0.035mm 0.035mm 0.035mm 0.035mm"/>
 <param name="mtIsolate" value="1.5mm 0.15mm 0.2mm 0.15mm 0.2mm 0.15mm 0.2mm 0.15mm 0.2mm 0.15mm 0.2mm 0.15mm 0.2mm 0.15mm 0.2mm"/>
-<param name="mdWireWire" value="6mil"/>
-<param name="mdWirePad" value="6mil"/>
-<param name="mdWireVia" value="6mil"/>
-<param name="mdPadPad" value="6mil"/>
-<param name="mdPadVia" value="6mil"/>
-<param name="mdViaVia" value="6mil"/>
-<param name="mdSmdPad" value="6mil"/>
-<param name="mdSmdVia" value="6mil"/>
-<param name="mdSmdSmd" value="6mil"/>
-<param name="mdViaViaSameLayer" value="6mil"/>
+<param name="mdWireWire" value="8mil"/>
+<param name="mdWirePad" value="8mil"/>
+<param name="mdWireVia" value="8mil"/>
+<param name="mdPadPad" value="8mil"/>
+<param name="mdPadVia" value="8mil"/>
+<param name="mdViaVia" value="8mil"/>
+<param name="mdSmdPad" value="8mil"/>
+<param name="mdSmdVia" value="8mil"/>
+<param name="mdSmdSmd" value="8mil"/>
+<param name="mdViaViaSameLayer" value="8mil"/>
 <param name="mnLayersViaInSmd" value="2"/>
-<param name="mdCopperDimension" value="40mil"/>
-<param name="mdDrill" value="6mil"/>
+<param name="mdCopperDimension" value="10mil"/>
+<param name="mdDrill" value="8mil"/>
 <param name="mdSmdStop" value="0mil"/>
-<param name="msWidth" value="6mil"/>
-<param name="msDrill" value="0.35mm"/>
+<param name="msWidth" value="8mil"/>
+<param name="msDrill" value="20mil"/>
 <param name="msMicroVia" value="9.99mm"/>
 <param name="msBlindViaRatio" value="0.5"/>
@@
 <param name="rvMicroViaOuter" value="0.25"/>
 <param name="rvMicroViaInner" value="0.25"/>
-<param name="rlMinPadTop" value="10mil"/>
+<param name="rlMinPadTop" value="12mil"/>
 <param name="rlMaxPadTop" value="20mil"/>
 <param name="rlMinPadInner" value="10mil"/>
 <param name="rlMaxPadInner" value="20mil"/>
-<param name="rlMinPadBottom" value="10mil"/>
+<param name="rlMinPadBottom" value="12mil"/>
 <param name="rlMaxPadBottom" value="20mil"/>
-<param name="rlMinViaOuter" value="8mil"/>
+<param name="rlMinViaOuter" value="10mil"/>
 <param name="rlMaxViaOuter" value="20mil"/>
-<param name="rlMinViaInner" value="8mil"/>
+<param name="rlMinViaInner" value="10mil"/>
 <param name="rlMaxViaInner" value="20mil"/>
 <param name="rlMinMicroViaOuter" value="4mil"/>
@@
 <param name="mlMinCreamFrame" value="0mil"/>
 <param name="mlMaxCreamFrame" value="0mil"/>
-<param name="mlViaStopLimit" value="0mil"/>
+<param name="mlViaStopLimit" value="25mil"/>
 <param name="srRoundness" value="0"/>
 <param name="srMinRoundness" value="0mil"/>

Commit message: POWER - DC DC 90% done.
Parts:
- added C1: 1u, rcl:C0805
- added C2, C3: ECA-1VM102B, IowaFormula:CAP_PAN_12.5X20
- added F1: 0505030.MXEP, IowaFormula:0505030.MXEP
- added J3, J4: 2P_1-770166-0, con-MATE-N-LOK:CON2_1X2_P163_VMNL-1MTG
- added R1: PWR221T-30-1R00F, IowaFormula:BO_PWR221T
- added U$1: DCMHEATSINK, IowaFormula:DCMHEATSINK
- added U$2: SRP1238A-R22M, IowaFormula:SRP1238A-R22M
- added U$3: SRP1238A-4R7M, IowaFormula:SRP1238A-R22M
- added X1, X2, X3, X4: 5566-2, con-molex:5566-2
- moved PS1 18.2 mm to (52.1, 52.1)
Connections:
- new net +12V-ISO: X1.1, X1.2, X2.1, X2.2
- new net +12V-OUT: C1.1, C2.1, C3.1, PS1.A2, R1.1, U$2.1
- new net GND: C1.2, C2.2, C3.2, PS1.B2, X3.1, X3.2, X4.1, X4.2
- new net HV+: F1.1, J3.1, J3.2
- new net HV+_IN: PS1.A1, U$3.2
- new net HV+_POSTFUSE: F1.2, U$3.1
- new net HV-: J4.1, J4.2, PS1.E1
- new net N$1: R1.2, U$2.2
Routing:
- net HV-: track 0.00 -> 56.5 mm
- net GND: track 0.00 -> 53.2 mm
- net +12V-OUT: track 0.00 -> 47.1 mm, vias 0 -> 1
- net +12V-ISO: track 0.00 -> 31.6 mm
- net HV+: track 0.00 -> 15.7 mm

Commit message: POWER - DCDC Rev A.
Parts:
- removed J3, J4: 2P_1-770166-0, con-MATE-N-LOK:CON2_1X2_P163_VMNL-1MTG
- removed U$2: SRP1238A-R22M, IowaFormula:SRP1238A-R22M
- removed X1, X3, X4: 5566-2, con-molex:5566-2
- added +12V-ISO1, .GND, >GND: 5566-2, con-molex:5566-2
- added C14, C4, C5, C7: ECA-2WHG2R2, IowaFormula:PCAP_10X125
- added HV+, HV-: 2P_1-770166-0, con-MATE-N-LOK:CON2_1X2_P163_VMNL-1MTG
- added R2: PWR221T-30-1R00F, IowaFormula:BO_PWR221T
- added U$4: SRP1238A-4R7M, IowaFormula:SRP1238A-R22M
- C1: value 1u -> ECA-2WHG2R2; device rcl:C0805 -> IowaFormula:PCAP_10X125
- moved C1 69.9 mm to (20.3, 25.4), turned to 0 degrees
- moved C3 51.4 mm to (94.0, 41.9), turned to 0 degrees
- moved C2 46.7 mm to (94.0, 55.9), turned to 0 degrees
- moved U$3 15.1 mm to (12.6, 54.5), turned to 180 degrees
- moved R1 11.4 mm to (66.0, 8.89), turned to 180 degrees
- moved F1 3.81 mm to (20.3, 72.4)
- renumbered X2 to +12V-ISO2
Connections:
- removed net HV+_IN: PS1.A1, U$3.2
- net +12V-ISO: now also +12V-ISO1.1, +12V-ISO1.2, C14.1, C5.1, R1.2, U$4.2; no longer X1.1, X1.2
- net +12V-OUT: now also U$4.1; no longer C1.1, U$2.1
- net GND: now also .GND.1, .GND.2, >GND.1, >GND.2, C14.2, C5.2; no longer C1.2, X3.1, X3.2, X4.1, X4.2
- net HV+: now also HV+.1, HV+.2; no longer J3.1, J3.2
- net HV+_POSTFUSE: now also R2.2
- net HV-: now also C1.2, C4.2, C7.2, HV-.1, HV-.2; no longer J4.1, J4.2
- net N$1: now also C1.1, C4.1, C7.1, PS1.A1, R2.1, U$3.2; no longer R1.2, U$2.2
Routing:
- net HV-: track 56.5 -> 4.14 mm
- net +12V-OUT: track 47.1 -> 0.00 mm, vias 1 -> 0
- net GND: track 53.2 -> 26.2 mm
- net HV+: track 15.7 -> 19.5 mm
- net +12V-ISO: track 31.6 -> 30.4 mm, vias 0 -> 1
- added copper zone on layer 1, net +12V-ISO
- added copper zone on layer 16, net +12V-ISO
- added copper zone on layer 1, net +12V-OUT
- added copper zone on layer 1, net GND
- added copper zone on layer 16, net GND
- added copper zone on layer 1, net HV+
- added copper zone on layer 1, net HV+_POSTFUSE
- added copper zone on layer 16, net HV-
- added copper zone on layer 1, net N$1
Other:
- board text added: "Author: github.com/michaelpass"
- board text added: "HV/Tractive System ~ 340VDC"
- board text added: "Iowa Formula"
- board text added: "Isolated DC-DC Converter POWER-DCDC Rev A: May 2nd, 2019"
