File: projects/PCB schematics/POWER/POWER-DCDC.brd (EAGLE design)
At the start: 99.1 x 99.1 mm, 20 parts

Commit message: POWER - DCDC changes w/ Ryan.
Parts:
- C7: value ECA-2WHG2R2 -> 2.2u
Changed lines of the file:
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@@
 </element>
 <element name="U$3" library="IowaFormula" package="SRP1238A-R22M" value="SRP1238A-4R7M" x="12.5984" y="54.4576" smashed="yes" rot="R180"/>
-<element name="C7" library="IowaFormula" package="PCAP_10X125" value="ECA-2WHG2R2" x="20.32" y="36.83" smashed="yes">
+<element name="C7" library="IowaFormula" package="PCAP_10X125" value="2.2u" x="20.32" y="36.83" smashed="yes">
 <attribute name="MANUFACTURER_PART_NUMBER" value="ECA2WHG2R2" x="20.32" y="36.83" size="1.778" layer="27" display="off"/>
 <attribute name="NAME" x="14.5542" y="36.195" size="1.27" layer="25" ratio="6" rot="SR0"/>

Commit message: PROJ - Final pre-purchase revisions (4 boards still in progress.)
Parts:
- renumbered +12V-ISO1 to +12V-ISO.1, +12V-ISO2 to +12V-ISO.2, .GND to GND.2, >GND to GND.1, PS1 to ISO-DCDC, U$1 to HEATSINK
Routing:
- added copper zone on layer 16, net HV+
Other:
- board text added: "Grounded Low Voltage System Peak: 12VDC"
- board text added: "HV/Tractive System Peak: 340VDC"
- board text removed: "HV/Tractive System ~ 340VDC"
Changed lines of the file:
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@@
 <dimension x1="37.1348" y1="15.0876" x2="62.7634" y2="14.9606" x3="49.9491" y3="24.1808" textsize="1.778" layer="21" dtype="horizontal" visible="yes"/>
 <text x="8.7884" y="13.8684" size="1.6764" layer="21" rot="R90">HV/Tractive System
-~ 340VDC </text>
+Peak: 340VDC </text>
+<text x="82.4484" y="13.8684" size="1.6764" layer="21" rot="R90">Grounded Low Voltage System
+Peak: 12VDC</text>
 </plain>
 <attributes>
@@
 </autorouter>
 <elements>
-<element name="PS1" library="DCM4623" package="DCM4623TD2N17C8T70" value="DCM4623TD2K31E0M70" x="52.07" y="52.07" smashed="yes">
+<element name="ISO-DCDC" library="DCM4623" package="DCM4623TD2N17C8T70" value="DCM4623TD2K31E0M70" x="52.07" y="52.07" smashed="yes">
 <attribute name="DESCRIPTION" value="Isolated DC/DC Converters 500W 270Vin 28Vout 4623 Package" x="52.07" y="52.07" size="1.778" layer="27" display="off"/>
 <attribute name="HEIGHT" value="5mm" x="52.07" y="52.07" size="1.778" layer="27" display="off"/>
@@
 <attribute name="VALUE" x="52.07" y="52.07" size="1.27" layer="27" align="center"/>
 </element>
-<element name="+12V-ISO1" library="con-molex" library_urn="urn:adsk.eagle:library:165" package="5566-2" package3d_urn="urn:adsk.eagle:package:8078583/1" value="5566-2" x="91.44" y="69.85" smashed="yes" rot="R270">
+<element name="+12V-ISO.1" library="con-molex" library_urn="urn:adsk.eagle:library:165" package="5566-2" package3d_urn="urn:adsk.eagle:package:8078583/1" value="5566-2" x="91.44" y="69.85" smashed="yes" rot="R270">
 <attribute name="MF" value="MOLEX" x="91.44" y="69.85" size="1.778" layer="27" rot="R270" display="off"/>
 <attribute name="MPN" value="" x="91.44" y="69.85" size="1.778" layer="27" rot="R270" display="off"/>
@@
 <attribute name="VALUE" x="85.09" y="72.39" size="1.27" layer="27" rot="R270"/>
 </element>
-<element name="+12V-ISO2" library="con-molex" library_urn="urn:adsk.eagle:library:165" package="5566-2" package3d_urn="urn:adsk.eagle:package:8078583/1" value="5566-2" x="91.44" y="83.82" smashed="yes" rot="R270">
+<element name="+12V-ISO.2" library="con-molex" library_urn="urn:adsk.eagle:library:165" package="5566-2" package3d_urn="urn:adsk.eagle:package:8078583/1" value="5566-2" x="91.44" y="83.82" smashed="yes" rot="R270">
 <attribute name="MF" value="MOLEX" x="91.44" y="83.82" size="1.778" layer="27" rot="R270" display="off"/>
 <attribute name="MPN" value="" x="91.44" y="83.82" size="1.778" layer="27" rot="R270" display="off"/>
@@
 <attribute name="VENDOR" value="TE Connectivity" x="35.56" y="5.08" size="1.778" layer="27" rot="R90" display="off"/>
 </element>
-<element name="&gt;GND" library="con-molex" library_urn="urn:adsk.eagle:library:165" package="5566-2" package3d_urn="urn:adsk.eagle:package:8078583/1" value="5566-2" x="91.44" y="30.48" smashed="yes" rot="R270">
+<element name="GND.1" library="con-molex" library_urn="urn:adsk.eagle:library:165" package="5566-2" package3d_urn="urn:adsk.eagle:package:8078583/1" value="5566-2" x="91.44" y="30.48" smashed="yes" rot="R270">
 <attribute name="MF" value="MOLEX" x="91.44" y="30.48" size="1.778" layer="27" rot="R270" display="off"/>
 <attribute name="MPN" value="" x="91.44" y="30.48" size="1.778" layer="27" rot="R270" display="off"/>
@@
 <attribute name="VALUE" x="85.09" y="33.02" size="1.27" layer="27" rot="R270"/>
 </element>
-<element name=".GND" library="con-molex" library_urn="urn:adsk.eagle:library:165" package="5566-2" package3d_urn="urn:adsk.eagle:package:8078583/1" value="5566-2" x="91.44" y="15.24" smashed="yes" rot="R270">
+<element name="GND.2" library="con-molex" library_urn="urn:adsk.eagle:library:165" package="5566-2" package3d_urn="urn:adsk.eagle:package:8078583/1" value="5566-2" x="91.44" y="15.24" smashed="yes" rot="R270">
 <attribute name="MF" value="MOLEX" x="91.44" y="15.24" size="1.778" layer="27" rot="R270" display="off"/>
 <attribute name="MPN" value="" x="91.44" y="15.24" size="1.778" layer="27" rot="R270" display="off"/>
@@
 <attribute name="VALUE" x="12.7" y="71.0946" size="1.778" layer="27" ratio="10" rot="R270"/>
 </element>
-<element name="U$1" library="IowaFormula" package="DCMHEATSINK" value="DCMHEATSINK" x="52.07" y="52.07" smashed="yes">
-<attribute name="NAME" x="52.07" y="48.26" size="1.27" layer="25" align="center"/>
+<element name="HEATSINK" library="IowaFormula" package="DCMHEATSINK" value="DCMHEATSINK" x="52.07" y="52.07" smashed="yes">
+<attribute name="NAME" x="52.07" y="38.1" size="1.27" layer="25" align="center"/>
 </element>
 <element name="R1" library="IowaFormula" package="BO_PWR221T" value="PWR221T-30-1R00F" x="66.04" y="8.89" smashed="yes" rot="R180">
@@
 <signals>
 <signal name="HV-">
-<contactref element="PS1" pad="E1"/>
+<contactref element="ISO-DCDC" pad="E1"/>
 <contactref element="HV-" pad="1"/>
 <contactref element="HV-" pad="2"/>
@@
 <vertex x="36.7538" y="45.6184"/>
 <vertex x="27.9908" y="45.6184"/>
-<vertex x="19.177" y="36.8046"/>
-<vertex x="19.177" y="2.5654"/>
+<vertex x="19.5834" y="37.211"/>
+<vertex x="19.5834" y="2.5654"/>
 <vertex x="36.7538" y="2.5654"/>
 </polygon>
 </signal>
 <signal name="+12V-ISO">
-<contactref element="+12V-ISO1" pad="1"/>
-<contactref element="+12V-ISO1" pad="2"/>
-<contactref element="+12V-ISO2" pad="1"/>
-<contactref element="+12V-ISO2" pad="2"/>
+<contactref element="+12V-ISO.1" pad="1"/>
+<contactref element="+12V-ISO.1" pad="2"/>
+<contactref element="+12V-ISO.2" pad="1"/>
+<contactref element="+12V-ISO.2" pad="2"/>
 <wire x1="88.69" y1="69.85" x2="94.19" y2="69.85" width="2.54" layer="1"/>
 <wire x1="88.69" y1="83.82" x2="94.19" y2="83.82" width="2.54" layer="1"/>
@@
 <vertex x="68.7578" y="37.2364"/>
 </polygon>
+<polygon width="0.254" layer="16" isolate="0.4064" thermals="no">
+<vertex x="67.31" y="87.63"/>
+<vertex x="68.58" y="86.36"/>
+<vertex x="86.36" y="86.36"/>
+<vertex x="86.36" y="81.28"/>
+<vertex x="96.52" y="81.28"/>
+<vertex x="96.52" y="96.52"/>
+<vertex x="67.31" y="96.52"/>
+</polygon>
 </signal>
 <signal name="GND">
-<contactref element="&gt;GND" pad="1"/>
-<contactref element="&gt;GND" pad="2"/>
-<contactref element=".GND" pad="1"/>
-<contactref element=".GND" pad="2"/>
+<contactref element="GND.1" pad="1"/>
+<contactref element="GND.1" pad="2"/>
+<contactref element="GND.2" pad="1"/>
+<contactref element="GND.2" pad="2"/>
 <wire x1="88.69" y1="30.48" x2="94.19" y2="30.48" width="2.54" layer="1"/>
 <wire x1="88.69" y1="15.24" x2="88.69" y2="30.48" width="2.54" layer="1"/>
-<contactref element="PS1" pad="B2"/>
+<contactref element="ISO-DCDC" pad="B2"/>
 <wire x1="88.69" y1="15.24" x2="94.19" y2="15.24" width="2.54" layer="1"/>
 <contactref element="C2" pad="2"/>
@@
 <vertex x="37.6682" y="79.6544"/>
 </polygon>
+<polygon width="0.254" layer="16" thermals="no">
+<vertex x="2.54" y="77.47"/>
+<vertex x="38.1" y="77.47"/>
+<vertex x="38.1" y="96.52"/>
+<vertex x="2.54" y="96.52"/>
+</polygon>
 </signal>
 <signal name="+12V-OUT">
-<contactref element="PS1" pad="A2"/>
+<contactref element="ISO-DCDC" pad="A2"/>
 <contactref element="R1" pad="1"/>
 <contactref element="C2" pad="1"/>
@@
 <contactref element="U$3" pad="2"/>
 <contactref element="C7" pad="1"/>
-<contactref element="PS1" pad="A1"/>
+<contactref element="ISO-DCDC" pad="A1"/>
 <contactref element="C1" pad="1"/>
 <contactref element="C4" pad="1"/>

Commit message: PROJ - Gerber files major milestone - 05/05/19.
Parts:
- U$3, U$4: value SRP1238A-4R7M -> SRP1238A-1R0M
Routing:
- added copper zone on layer 16, net HV+_POSTFUSE
- added copper zone on layer 1, net HV-
- added copper zone on layer 16, net N$1
Other:
- board text added: "Isolated DC-DC Converter POWER-DCDC Rev A: May 5th, 2019"
- board text removed: "Isolated DC-DC Converter POWER-DCDC Rev A: May 2nd, 2019"
Changed lines of the file:
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@@
 <text x="42.0624" y="6.8834" size="1.016" layer="25" font="vector">Isolated DC-DC Converter
 POWER-DCDC
-Rev A: May 2nd, 2019</text>
+Rev A: May 5th, 2019</text>
 <text x="66.8528" y="2.4384" size="1.016" layer="25" font="vector">Author: github.com/michaelpass</text>
 <wire x1="37.0332" y1="97.8154" x2="37.0332" y2="1.2954" width="0.4064" layer="21" style="shortdash"/>
@@
 <attribute name="VENDOR" value="Bourns Electronics" x="66.04" y="8.89" size="1.778" layer="27" rot="R180" display="off"/>
 </element>
-<element name="U$3" library="IowaFormula" package="SRP1238A-R22M" value="SRP1238A-4R7M" x="12.5984" y="54.4576" smashed="yes" rot="R180"/>
+<element name="U$3" library="IowaFormula" package="SRP1238A-R22M" value="SRP1238A-1R0M" x="12.5984" y="54.4576" smashed="yes" rot="R180"/>
 <element name="C7" library="IowaFormula" package="PCAP_10X125" value="2.2u" x="20.32" y="36.83" smashed="yes">
 <attribute name="MANUFACTURER_PART_NUMBER" value="ECA2WHG2R2" x="20.32" y="36.83" size="1.778" layer="27" display="off"/>
@@
 <attribute name="VENDOR" value="Panasonic" x="79.4512" y="82.6516" size="1.778" layer="27" rot="R270" display="off"/>
 </element>
-<element name="U$4" library="IowaFormula" package="SRP1238A-R22M" value="SRP1238A-4R7M" x="73.66" y="17.78" smashed="yes" rot="R180"/>
+<element name="U$4" library="IowaFormula" package="SRP1238A-R22M" value="SRP1238A-1R0M" x="73.66" y="17.78" smashed="yes" rot="R180"/>
 <element name="C1" library="IowaFormula" package="PCAP_10X125" value="ECA-2WHG2R2" x="20.32" y="25.4" smashed="yes">
 <attribute name="MANUFACTURER_PART_NUMBER" value="ECA2WHG2R2" x="20.32" y="25.4" size="1.778" layer="27" display="off"/>
@@
 <vertex x="36.7538" y="45.6184"/>
 <vertex x="27.9908" y="45.6184"/>
-<vertex x="19.5834" y="37.211"/>
-<vertex x="19.5834" y="2.5654"/>
+<vertex x="19.6088" y="37.2364"/>
+<vertex x="19.6088" y="2.5654"/>
 <vertex x="36.7538" y="2.5654"/>
+</polygon>
+<polygon width="0.254" layer="1" isolate="0.8128" thermals="no">
+<vertex x="19.9136" y="37.6428"/>
+<vertex x="36.83" y="37.6428"/>
+<vertex x="36.83" y="2.54"/>
+<vertex x="19.9136" y="2.54"/>
 </polygon>
 </signal>
@@
 <contactref element="R2" pad="2"/>
 <polygon width="0.3048" layer="1" isolate="1.27" thermals="no">
-<vertex x="9.2964" y="44.196"/>
-<vertex x="12.0396" y="41.4528"/>
+<vertex x="9.525" y="44.3484"/>
+<vertex x="12.4206" y="41.4528"/>
 <vertex x="24.3586" y="41.4528"/>
 <vertex x="24.3586" y="56.2864"/>
 <vertex x="18.923" y="61.722"/>
 <vertex x="12.8016" y="61.722"/>
-<vertex x="9.2964" y="58.2168"/>
+<vertex x="9.525" y="58.4454"/>
+</polygon>
+<polygon width="0.254" layer="16" isolate="0.4064" thermals="no">
+<vertex x="9.7536" y="57.15"/>
+<vertex x="9.7536" y="43.7134"/>
+<vertex x="18.5674" y="43.7134"/>
+<vertex x="24.3332" y="49.4792"/>
+<vertex x="21.59" y="52.2224"/>
+<vertex x="21.59" y="55.88"/>
+<vertex x="20.32" y="57.15"/>
 </polygon>
 </signal>
@@
 <vertex x="11.9634" y="37.6428"/>
 </polygon>
-</signal>
+<polygon width="0.254" layer="16" isolate="0.4064" thermals="no">
+<vertex x="15.9258" y="2.54"/>
+<vertex x="15.9258" y="38.1"/>
+<vertex x="11.43" y="38.1"/>
+<vertex x="5.6896" y="43.8404"/>
+<vertex x="5.6896" y="60.7822"/>
+<vertex x="10.4902" y="65.5828"/>
+<vertex x="22.0218" y="65.5828"/>
+<vertex x="22.0218" y="73.1012"/>
+<vertex x="21.971" y="73.152"/>
+<vertex x="0.9906" y="73.152"/>
+<vertex x="0.889" y="73.2536"/>
+<vertex x="0.889" y="2.667"/>
+<vertex x="1.016" y="2.54"/>
+</polygon>
+</signal>
