File: projects/PCB schematics/POWER/POWER-12V5V.sch (EAGLE design)
At the start: 23 parts, among them U1 UCC383TDKTTT-5, U2 UCC383TDKTTT-5, U3 UCC383TDKTTT-5, X1 5566-2, X2 5566-2, X3 5566-2, X4 5566-2, X5 5566-2

Commit message: POWER - 12V5V revisions.
Parts:
- added X11, X6, X7, X9: 5566-2, con-molex:5566-2
Connections:
- net +12V-ISO: now also X6-1.S, X6-2.S
- net +5V: now also X9-1.S, X9-2.S
- net GND: now also X11-1.S, X11-2.S
- net VCC: now also X7-1.S, X7-2.S
Other:
- moved on the sheet: C1, C10, C11, C12, C2, C3, C4, C5, C6, C7, C8, C9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

Commit message: POWER - 12V5V Rev A.
Parts:
- removed X1, X11, X2, X3, X4, X5, X6, X7, X9: 5566-2, con-molex:5566-2
- added +12V-ISO.1, +12V-ISO.2, +5V.1, +5V.2, GND.1, GND.2, GND.3, VCC.1, VCC.2: 5566-2, con-molex:5566-2
- added C13, C14, C15: 100n, rcl:C-USC0805
- C10, C12, C9: value (none) -> 1u
Connections:
- removed net N$1: C4.+, C9.1, U1.VOUT
- removed net N$2: C11.+, C12.1, U3.VOUT
- removed net N$3: C10.1, C6.+, U2.VOUT
- net +12V-ISO: now also +12V-ISO.1-1.S, +12V-ISO.1-2.S, +12V-ISO.2-1.S, +12V-ISO.2-2.S; no longer X1-1.S, X1-2.S, X6-1.S, X6-2.S
- net +5V: now also +5V.1-1.S, +5V.1-2.S, +5V.2-1.S, +5V.2-2.S; no longer X3-1.S, X3-2.S, X9-1.S, X9-2.S
- net GND: now also C13.2, C14.2, C15.2, GND.1-1.S, GND.1-2.S, GND.2-1.S, GND.2-2.S, GND.3-1.S, GND.3-2.S; no longer X11-1.S, X11-2.S, X2-1.S, X2-2.S, X5-1.S, X5-2.S
- net VCC: now also C10.1, C11.+, C12.1, C13.1, C14.1, C15.1, C4.+, C6.+, C9.1, U1.VOUT, U2.VOUT, U3.VOUT, VCC.1-1.S, VCC.1-2.S, VCC.2-1.S, VCC.2-2.S; no longer X4-1.S, X4-2.S, X7-1.S, X7-2.S
Other:
- note added: "Note: TTL logic boards (vehicle control boards) should normally be hooked up to VCC. +5V is the output from the +12V converter, and if this is too high, 5V TTL logic may be used out of spec. By default, hook up +5V access to VCC. If underpowered, or voltage drops too low (drop-out voltage of 5V LDO linear regulator changes with current draw), switch to +5V."
- moved on the sheet: C1, C10, C11, C12, C2, C3, C4, C5, C6, C7, C8, C9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
