File: projects/PCB schematics/RTDS/RTDS.brd (EAGLE design)
At the start: 99.1 x 99.1 mm, 11 parts, among them X1 5566-2, X2 5566-2, X3 5566-2, X4 5566-2, X5 5566-2

Commit message: PROJ - Final pre-purchase revisions (4 boards still in progress.)
Parts:
- renumbered X1 to +12V-ISO.1, X2 to +12V-ISO.2, X3 to VCC.1, X4 to GND.1, X5 to RTDS_SIGNAL
Other:
- board text added: "- Connect +12V-ISO.2 pins to 12V power terminals on MAX9744 - Connect speakers to R/L terminal output block son MAX9744"
- board text added: "I/O: 1. RTDS_SIGNAL 2. VCC.1 3. GND 4. +12V-ISO (X1) 5. +12V-ISO (X2)"
- board text removed: "I/O: 1. +12V-ISO (X1) 2. +12V-ISO (X2) 3. VCC (X3) 4. GND (X4) 5. RTDS_SIGNAL (X5)"
Changed lines of the file:
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@@
 <setting verticaltext="up"/>
 </settings>
-<grid distance="3.125" unitdist="mil" unit="mil" style="lines" multiple="1" display="yes" altdistance="1" altunitdist="mil" altunit="mil"/>
+<grid distance="50" unitdist="mil" unit="mil" style="lines" multiple="1" display="yes" altdistance="1" altunitdist="mil" altunit="mil"/>
 <layers>
 <layer number="1" name="Top" color="4" fill="1" visible="yes" active="yes"/>
@@
 <text x="86.36" y="15.24" size="1.016" layer="25" rot="R90">Author: github.com/michaelpass</text>
 <text x="36.7284" y="71.2216" size="1.27" layer="25">I/O:
-1. +12V-ISO (X1)
-2. +12V-ISO (X2)
-3. VCC (X3)
-4. GND (X4)
-5. RTDS_SIGNAL (X5)</text>
-<dimension x1="62.6618" y1="85.7504" x2="49.5554" y2="85.7504" x3="56.1086" y3="83.9978" textsize="1.778" layer="1"/>
+1. RTDS_SIGNAL
+2. VCC.1
+3. GND
+4. +12V-ISO (X1)
+5. +12V-ISO (X2)</text>
+<text x="36.83" y="16.51" size="1.016" layer="21" rot="R90">- Connect +12V-ISO.2 pins to 12V power terminals on MAX9744
+- Connect speakers to R/L terminal output block son MAX9744</text>
 </plain>
 <attributes>
@@
 <attribute name="VALUE" x="60.96" y="66.675" size="1.27" layer="27"/>
 </element>
-<element name="X3" library="con-molex" library_urn="urn:adsk.eagle:library:165" package="5566-2" package3d_urn="urn:adsk.eagle:package:8078583/1" value="5566-2" x="29.21" y="91.44" smashed="yes">
+<element name="VCC.1" library="con-molex" library_urn="urn:adsk.eagle:library:165" package="5566-2" package3d_urn="urn:adsk.eagle:package:8078583/1" value="5566-2" x="29.21" y="91.44" smashed="yes">
 <attribute name="MF" value="MOLEX" x="29.21" y="91.44" size="1.778" layer="27" display="off"/>
 <attribute name="MPN" value="" x="29.21" y="91.44" size="1.778" layer="27" display="off"/>
-<attribute name="NAME" x="27.94" y="96.52" size="1.27" layer="25"/>
+<attribute name="NAME" x="26.67" y="96.52" size="1.27" layer="25"/>
 <attribute name="OC_FARNELL" value="1822072" x="29.21" y="91.44" size="1.778" layer="27" display="off"/>
 <attribute name="OC_NEWARK" value="unknown" x="29.21" y="91.44" size="1.778" layer="27" display="off"/>
 <attribute name="VALUE" x="26.67" y="85.09" size="1.27" layer="27"/>
 </element>
-<element name="X4" library="con-molex" library_urn="urn:adsk.eagle:library:165" package="5566-2" package3d_urn="urn:adsk.eagle:package:8078583/1" value="5566-2" x="44.45" y="91.44" smashed="yes">
+<element name="GND.1" library="con-molex" library_urn="urn:adsk.eagle:library:165" package="5566-2" package3d_urn="urn:adsk.eagle:package:8078583/1" value="5566-2" x="44.45" y="91.44" smashed="yes">
 <attribute name="MF" value="MOLEX" x="44.45" y="91.44" size="1.778" layer="27" display="off"/>
 <attribute name="MPN" value="" x="44.45" y="91.44" size="1.778" layer="27" display="off"/>
-<attribute name="NAME" x="43.18" y="96.52" size="1.27" layer="25"/>
+<attribute name="NAME" x="41.91" y="96.52" size="1.27" layer="25"/>
 <attribute name="OC_FARNELL" value="1822072" x="44.45" y="91.44" size="1.778" layer="27" display="off"/>
 <attribute name="OC_NEWARK" value="unknown" x="44.45" y="91.44" size="1.778" layer="27" display="off"/>
 <attribute name="VALUE" x="41.91" y="85.09" size="1.27" layer="27"/>
 </element>
-<element name="X5" library="con-molex" library_urn="urn:adsk.eagle:library:165" package="5566-2" package3d_urn="urn:adsk.eagle:package:8078583/1" value="5566-2" x="13.97" y="91.44" smashed="yes">
+<element name="RTDS_SIGNAL" library="con-molex" library_urn="urn:adsk.eagle:library:165" package="5566-2" package3d_urn="urn:adsk.eagle:package:8078583/1" value="5566-2" x="13.97" y="91.44" smashed="yes">
 <attribute name="MF" value="MOLEX" x="13.97" y="91.44" size="1.778" layer="27" display="off"/>
 <attribute name="MPN" value="" x="13.97" y="91.44" size="1.778" layer="27" display="off"/>
-<attribute name="NAME" x="12.7" y="96.52" size="1.27" layer="25"/>
+<attribute name="NAME" x="8.255" y="96.440625" size="1.27" layer="25"/>
 <attribute name="OC_FARNELL" value="1822072" x="13.97" y="91.44" size="1.778" layer="27" display="off"/>
 <attribute name="OC_NEWARK" value="unknown" x="13.97" y="91.44" size="1.778" layer="27" display="off"/>
@@
 <attribute name="NAME" x="62.992" y="85.09" size="1.27" layer="25" ratio="16" rot="R90"/>
 </element>
-<element name="X2" library="con-molex" library_urn="urn:adsk.eagle:library:165" package="5566-2" package3d_urn="urn:adsk.eagle:package:8078583/1" value="5566-2" x="29.21" y="74.93" smashed="yes">
+<element name="+12V-ISO.2" library="con-molex" library_urn="urn:adsk.eagle:library:165" package="5566-2" package3d_urn="urn:adsk.eagle:package:8078583/1" value="5566-2" x="29.21" y="74.93" smashed="yes">
 <attribute name="MF" value="MOLEX" x="29.21" y="74.93" size="1.778" layer="27" display="off"/>
 <attribute name="MPN" value="" x="29.21" y="74.93" size="1.778" layer="27" display="off"/>
-<attribute name="NAME" x="27.94" y="80.01" size="1.27" layer="25"/>
+<attribute name="NAME" x="25.4" y="80.01" size="1.27" layer="25"/>
 <attribute name="OC_FARNELL" value="1822072" x="29.21" y="74.93" size="1.778" layer="27" display="off"/>
 <attribute name="OC_NEWARK" value="unknown" x="29.21" y="74.93" size="1.778" layer="27" display="off"/>
@@
 </element>
 <element name="U$3" library="IowaFormula" package="MAX9744" value="MAX9744" x="2.54" y="60.96" smashed="yes" rot="R270">
-<attribute name="VALUE" x="-0.635" y="54.61" size="1.27" layer="27" rot="R270"/>
+<attribute name="VALUE" x="41.275" y="34.29" size="1.27" layer="27" rot="R270"/>
 </element>
 <element name="R1" library="rcl" library_urn="urn:adsk.eagle:library:334" package="R0805" package3d_urn="urn:adsk.eagle:package:23553/2" value="47k" x="21.1328" y="88.6206" smashed="yes" rot="R180">
@@
 <attribute name="VALUE" x="50.165" y="63.5" size="1.27" layer="27"/>
 </element>
-<element name="X1" library="con-molex" library_urn="urn:adsk.eagle:library:165" package="5566-2" package3d_urn="urn:adsk.eagle:package:8078583/1" value="5566-2" x="13.97" y="74.93" smashed="yes">
+<element name="+12V-ISO.1" library="con-molex" library_urn="urn:adsk.eagle:library:165" package="5566-2" package3d_urn="urn:adsk.eagle:package:8078583/1" value="5566-2" x="13.97" y="74.93" smashed="yes">
 <attribute name="MF" value="MOLEX" x="1.27" y="88.9" size="1.778" layer="27" display="off"/>
 <attribute name="MPN" value="" x="1.27" y="88.9" size="1.778" layer="27" display="off"/>
-<attribute name="NAME" x="12.7" y="80.01" size="1.27" layer="25"/>
+<attribute name="NAME" x="10.16" y="80.01" size="1.27" layer="25"/>
 <attribute name="OC_FARNELL" value="1822072" x="1.27" y="88.9" size="1.778" layer="27" display="off"/>
 <attribute name="OC_NEWARK" value="unknown" x="1.27" y="88.9" size="1.778" layer="27" display="off"/>
@@
 </signal>
 <signal name="GND">
-<contactref element="X4" pad="1"/>
-<contactref element="X4" pad="2"/>
+<contactref element="GND.1" pad="1"/>
+<contactref element="GND.1" pad="2"/>
 <contactref element="U$2" pad="11"/>
 <polygon width="0.6096" layer="1" isolate="0.3048">
@@
 </signal>
 <signal name="VCC">
-<contactref element="X3" pad="1"/>
-<contactref element="X3" pad="2"/>
+<contactref element="VCC.1" pad="1"/>
+<contactref element="VCC.1" pad="2"/>
 <contactref element="SH1" pad="2"/>
 <contactref element="R1" pad="1"/>
@@
 <via x="47.879" y="66.04" extent="1-16" drill="0.508"/>
 <wire x1="47.879" y1="66.04" x2="49.85" y2="66.04" width="0.6096" layer="1"/>
-<wire x1="37.995" y1="79.905" x2="42.2402" y2="84.1502" width="0.6096" layer="16"/>
-<wire x1="42.2402" y1="84.1502" x2="60.96" y2="84.1502" width="0.6096" layer="16"/>
-<via x="60.96" y="84.1502" extent="1-16" drill="0.508"/>
-<wire x1="60.96" y1="84.1502" x2="60.96" y2="85.725" width="0.6096" layer="1"/>
+<wire x1="37.995" y1="79.905" x2="41.1988" y2="83.1088" width="0.6096" layer="16"/>
+<wire x1="60.4774" y1="83.1088" x2="60.9854" y2="83.6168" width="0.6096" layer="16"/>
+<wire x1="60.4774" y1="83.1088" x2="41.1988" y2="83.1088" width="0.6096" layer="16"/>
+<via x="60.9854" y="83.6168" extent="1-16" drill="0.508"/>
+<wire x1="60.9854" y1="85.6996" x2="60.9854" y2="83.6168" width="0.6096" layer="1"/>
+<wire x1="60.9854" y1="85.6996" x2="60.96" y2="85.725" width="0.6096" layer="1"/>
 </signal>
 <signal name="RTDS_SIGNAL">
-<contactref element="X5" pad="1"/>
-<contactref element="X5" pad="2"/>
+<contactref element="RTDS_SIGNAL" pad="1"/>
+<contactref element="RTDS_SIGNAL" pad="2"/>
 <contactref element="U$2" pad="2"/>
 <contactref element="R1" pad="2"/>
@@
 </signal>
 <signal name="+12V-ISO">
-<contactref element="X2" pad="1"/>
-<contactref element="X2" pad="2"/>
-<contactref element="X1" pad="1"/>
-<contactref element="X1" pad="2"/>
+<contactref element="+12V-ISO.2" pad="1"/>
+<contactref element="+12V-ISO.2" pad="2"/>
+<contactref element="+12V-ISO.1" pad="1"/>
+<contactref element="+12V-ISO.1" pad="2"/>
 <wire x1="13.97" y1="77.68" x2="13.97" y2="72.18" width="0.6096" layer="16"/>
 <wire x1="29.21" y1="77.68" x2="29.21" y2="72.18" width="0.6096" layer="16"/>

Commit message: PROJ - Gerber files major milestone - 05/05/19.
Connections:
- removed net N$1: U$1.GND
- net GND: now also U$1.GND
Other:
- board text added: "Rready-To-Drive Sound (RTDS) Board Rev A: May 5th, 2019"
- board text removed: "Rready-To-Drive Sound (RTDS) Board Rev A: 04/30/19"
Changed lines of the file:
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@@
 <hole x="91.44" y="95.25" drill="3"/>
 <text x="84.201" y="15.621" size="1.778" layer="25" font="vector" rot="R90">Rready-To-Drive Sound (RTDS) Board
-Rev A: 04/30/19</text>
+Rev A: May 5th, 2019</text>
 <wire x1="64.3128" y1="29.5402" x2="77.5208" y2="29.5402" width="0.1524" layer="25"/>
 <wire x1="77.5208" y1="29.5402" x2="77.5208" y2="43.5102" width="0.1524" layer="25"/>
@@
 <contactref element="GND.1" pad="2"/>
 <contactref element="U$2" pad="11"/>
-<polygon width="0.6096" layer="1" isolate="0.3048">
+<polygon width="0.6096" layer="1" isolate="0.4064">
 <vertex x="1.27" y="97.79"/>
 <vertex x="93.98" y="97.79"/>
@@
 <contactref element="U$2" pad="15"/>
 <contactref element="U$3" pad="GND"/>
+<contactref element="U$1" pad="GND"/>
 </signal>
 <signal name="VCC">
@@
 <wire x1="49.53" y1="81.28" x2="83.82" y2="81.28" width="0.6096" layer="1"/>
 </signal>
-<signal name="N$1">
-<contactref element="U$1" pad="GND"/>
-</signal>
 </signals>
