File: projects/PCB schematics/SC/SC-STAGE.sch (EAGLE design)
At the start: 0 parts

Commit message: SC - Stage initial placement.
Parts:
- added BSPD, BSPDPLAUS1, BSPDPLAUS2, IMD: (no value), con-lstb:MA03-1
- added LED1, LED2, LED3, LED4: 150080VS75000, 150080VS75000:150080VS75000
- added NOT1: 74LS19D, 74xx-us:74LS19D
- added Q1, Q2, Q3, Q4: IRLZ44Z, transistor-power:IRLZ44Z
- added R1, R10, R11, R12, R2, R3, R4, R9: (no value), rcl:R-US_R0805
- added R13, R14, R5, R6: 47k, rcl:R-US_R0805
- added R15, R16, R7, R8: 100, rcl:R-US_R0805
- added U1, U2, U3, U4: G5LE-1A-E-DC12, IowaFormula:G5LE-1A-E-DC12
- added X1, X3, X4, X5, X6: 5566-2, con-molex:5566-2
- added X2: 5566-4, con-molex:5566-4
Connections:
- new net +12V: U1.4, U2.4, U3.4, U4.4
- new net +12V-ISO: X1-1.S, X1-2.S
- new net BSPDFAULT_LED: BSPD.1, X2-1.S
- new net BSPDPLAUS1_LED: BSPDPLAUS1.1, X2-2.S
- new net BSPDPLAUS2_LED: BSPDPLAUS2.1, X2-3.S
- new net GND: BSPD.3, BSPDPLAUS1.3, BSPDPLAUS2.3, IMD.3, Q1.S, Q2.S, Q3.S, Q4.S, R11.1, R12.1, R13.1, R14.1, R3.1, R4.1, R5.1, R6.1, X5-1.S, X5-2.S
- new net IMDFAULT_LED: IMD.1, X2-4.S
- new net LED4: LED4.K, R11.2
- new net N$1: Q1.G, R7.2
- new net N$10: U3.2, U4.3
- new net N$105105: BSPD.2, NOT1A.I, R1.1
- new net N$11552: BSPDPLAUS1.2, NOT1B.I, R2.1
- new net N$14: Q4.G, R15.2
- new net N$15: LED4.A, NOT1D.O, R13.2, R15.1
- new net N$17: Q4.D, U4.1
- new net N$18: Q3.G, R16.2
- new net N$19: LED3.A, NOT1C.O, R14.2, R16.1
- new net N$2: LED1.A, NOT1A.O, R5.2, R7.1
- new net N$20: LED3.K, R12.2
- new net N$21: Q3.D, U3.1
- new net N$3: LED1.K, R3.2
- new net N$38: U2.2, U3.3
- new net N$4: Q1.D, U1.1
- new net N$5: Q2.G, R8.2
- new net N$6: LED2.A, NOT1B.O, R6.2, R8.1
- new net N$626: BSPDPLAUS2.2, NOT1C.I, R10.1
- new net N$7: LED2.K, R4.2
- new net N$8: Q2.D, U2.1
- new net N$9: U1.2, U2.3
- new net N$9581: IMD.2, NOT1D.I, R9.1
- new net SC+: U1.3, X4-1.S, X4-2.S
- new net SC-: U4.2, X6-1.S, X6-2.S
- new net VCC: R1.2, R10.2, R2.2, R9.2, X3-1.S, X3-2.S

Commit message: SC - SC-STAGE Rev. A
Parts:
- renumbered X1 to 12V-ISO, X3 to VCC, X4 to SC+, X5 to GND, X6 to SC-
Connections:
- removed net +12V: U1.4, U2.4, U3.4, U4.4
- net +12V-ISO: now also U1.4, U2.4, U3.4, U4.4
Changed lines of the file:
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@@
 </classes>
 <parts>
-<part name="X1" library="con-molex" library_urn="urn:adsk.eagle:library:165" deviceset="5566-2" device="" package3d_urn="urn:adsk.eagle:package:8078583/1"/>
-<part name="X3" library="con-molex" library_urn="urn:adsk.eagle:library:165" deviceset="5566-2" device="" package3d_urn="urn:adsk.eagle:package:8078583/1"/>
-<part name="X5" library="con-molex" library_urn="urn:adsk.eagle:library:165" deviceset="5566-2" device="" package3d_urn="urn:adsk.eagle:package:8078583/1"/>
-<part name="X4" library="con-molex" library_urn="urn:adsk.eagle:library:165" deviceset="5566-2" device="" package3d_urn="urn:adsk.eagle:package:8078583/1"/>
-<part name="X6" library="con-molex" library_urn="urn:adsk.eagle:library:165" deviceset="5566-2" device="" package3d_urn="urn:adsk.eagle:package:8078583/1"/>
+<part name="12V-ISO" library="con-molex" library_urn="urn:adsk.eagle:library:165" deviceset="5566-2" device="" package3d_urn="urn:adsk.eagle:package:8078583/1"/>
+<part name="VCC" library="con-molex" library_urn="urn:adsk.eagle:library:165" deviceset="5566-2" device="" package3d_urn="urn:adsk.eagle:package:8078583/1"/>
+<part name="GND" library="con-molex" library_urn="urn:adsk.eagle:library:165" deviceset="5566-2" device="" package3d_urn="urn:adsk.eagle:package:8078583/1"/>
+<part name="SC+" library="con-molex" library_urn="urn:adsk.eagle:library:165" deviceset="5566-2" device="" package3d_urn="urn:adsk.eagle:package:8078583/1"/>
+<part name="SC-" library="con-molex" library_urn="urn:adsk.eagle:library:165" deviceset="5566-2" device="" package3d_urn="urn:adsk.eagle:package:8078583/1"/>
 <part name="R7" library="rcl" library_urn="urn:adsk.eagle:library:334" deviceset="R-US_" device="R0805" package3d_urn="urn:adsk.eagle:package:23553/2" value="100"/>
 <part name="R5" library="rcl" library_urn="urn:adsk.eagle:library:334" deviceset="R-US_" device="R0805" package3d_urn="urn:adsk.eagle:package:23553/2" value="47k"/>
@@
 </plain>
 <instances>
-<instance part="X1" gate="-1" x="30.48" y="127" smashed="yes">
+<instance part="12V-ISO" gate="-1" x="30.48" y="127" smashed="yes">
 <attribute name="NAME" x="33.02" y="126.238" size="1.524" layer="95"/>
 <attribute name="VALUE" x="29.718" y="128.397" size="1.778" layer="96"/>
 </instance>
-<instance part="X1" gate="-2" x="30.48" y="121.92" smashed="yes">
+<instance part="12V-ISO" gate="-2" x="30.48" y="121.92" smashed="yes">
 <attribute name="NAME" x="33.02" y="121.158" size="1.524" layer="95"/>
 <attribute name="VALUE" x="29.718" y="123.317" size="1.778" layer="96"/>
 </instance>
-<instance part="X3" gate="-1" x="68.58" y="127" smashed="yes">
+<instance part="VCC" gate="-1" x="68.58" y="127" smashed="yes">
 <attribute name="NAME" x="71.12" y="126.238" size="1.524" layer="95"/>
 <attribute name="VALUE" x="67.818" y="128.397" size="1.778" layer="96"/>
 </instance>
-<instance part="X3" gate="-2" x="68.58" y="121.92" smashed="yes">
+<instance part="VCC" gate="-2" x="68.58" y="121.92" smashed="yes">
 <attribute name="NAME" x="71.12" y="121.158" size="1.524" layer="95"/>
 <attribute name="VALUE" x="67.818" y="123.317" size="1.778" layer="96"/>
 </instance>
-<instance part="X5" gate="-1" x="101.6" y="127" smashed="yes">
+<instance part="GND" gate="-1" x="101.6" y="127" smashed="yes">
 <attribute name="NAME" x="104.14" y="126.238" size="1.524" layer="95"/>
 <attribute name="VALUE" x="100.838" y="128.397" size="1.778" layer="96"/>
 </instance>
-<instance part="X5" gate="-2" x="101.6" y="121.92" smashed="yes">
+<instance part="GND" gate="-2" x="101.6" y="121.92" smashed="yes">
 <attribute name="NAME" x="104.14" y="121.158" size="1.524" layer="95"/>
 <attribute name="VALUE" x="100.838" y="123.317" size="1.778" layer="96"/>
 </instance>
-<instance part="X4" gate="-1" x="68.58" y="99.06" smashed="yes">
+<instance part="SC+" gate="-1" x="68.58" y="99.06" smashed="yes">
 <attribute name="NAME" x="71.12" y="98.298" size="1.524" layer="95"/>
 <attribute name="VALUE" x="67.818" y="100.457" size="1.778" layer="96"/>
 </instance>
-<instance part="X4" gate="-2" x="68.58" y="93.98" smashed="yes">
+<instance part="SC+" gate="-2" x="68.58" y="93.98" smashed="yes">
 <attribute name="NAME" x="71.12" y="93.218" size="1.524" layer="95"/>
 <attribute name="VALUE" x="67.818" y="95.377" size="1.778" layer="96"/>
 </instance>
-<instance part="X6" gate="-1" x="101.6" y="99.06" smashed="yes">
+<instance part="SC-" gate="-1" x="101.6" y="99.06" smashed="yes">
 <attribute name="NAME" x="104.14" y="98.298" size="1.524" layer="95"/>
 <attribute name="VALUE" x="100.838" y="100.457" size="1.778" layer="96"/>
 </instance>
-<instance part="X6" gate="-2" x="101.6" y="93.98" smashed="yes">
+<instance part="SC-" gate="-2" x="101.6" y="93.98" smashed="yes">
 <attribute name="NAME" x="104.14" y="93.218" size="1.524" layer="95"/>
 <attribute name="VALUE" x="100.838" y="95.377" size="1.778" layer="96"/>
@@
 <net name="GND" class="0">
 <segment>
-<pinref part="X5" gate="-1" pin="S"/>
+<pinref part="GND" gate="-1" pin="S"/>
 <wire x1="99.06" y1="127" x2="96.52" y2="127" width="0.1524" layer="91"/>
 <wire x1="96.52" y1="127" x2="86.36" y2="127" width="0.1524" layer="91"/>
 <wire x1="96.52" y1="127" x2="96.52" y2="121.92" width="0.1524" layer="91"/>
 <junction x="96.52" y="127"/>
-<pinref part="X5" gate="-2" pin="S"/>
+<pinref part="GND" gate="-2" pin="S"/>
 <wire x1="96.52" y1="121.92" x2="99.06" y2="121.92" width="0.1524" layer="91"/>
 <label x="86.36" y="127" size="1.778" layer="95"/>
@@
 <wire x1="25.4" y1="121.92" x2="27.94" y2="121.92" width="0.1524" layer="91"/>
 <label x="12.7" y="127" size="1.778" layer="95"/>
-<pinref part="X1" gate="-1" pin="S"/>
-<pinref part="X1" gate="-2" pin="S"/>
+<pinref part="12V-ISO" gate="-1" pin="S"/>
+<pinref part="12V-ISO" gate="-2" pin="S"/>
+</segment>
+<segment>
+<pinref part="P+4" gate="1" pin="+12V"/>
+<pinref part="U2" gate="A" pin="4"/>
+<wire x1="241.3" y1="109.22" x2="241.3" y2="106.68" width="0.1524" layer="91"/>
+</segment>
+<segment>
+<pinref part="P+3" gate="1" pin="+12V"/>
+<pinref part="U1" gate="A" pin="4"/>
+<wire x1="241.3" y1="210.82" x2="241.3" y2="208.28" width="0.1524" layer="91"/>
+</segment>
+<segment>
+<pinref part="P+8" gate="1" pin="+12V"/>
+<pinref part="U3" gate="A" pin="4"/>
+<wire x1="426.72" y1="213.36" x2="426.72" y2="210.82" width="0.1524" layer="91"/>
+</segment>
+<segment>
+<pinref part="P+7" gate="1" pin="+12V"/>
+<pinref part="U4" gate="A" pin="4"/>
+<wire x1="424.18" y1="109.22" x2="424.18" y2="106.68" width="0.1524" layer="91"/>
 </segment>
 </net>
@@
 <wire x1="63.5" y1="121.92" x2="66.04" y2="121.92" width="0.1524" layer="91"/>
 <label x="53.34" y="127" size="1.778" layer="95"/>
-<pinref part="X3" gate="-1" pin="S"/>
-<pinref part="X3" gate="-2" pin="S"/>
+<pinref part="VCC" gate="-1" pin="S"/>
+<pinref part="VCC" gate="-2" pin="S"/>
 </segment>
 <segment>
@@
 </segment>
 </net>
-<net name="+12V" class="0">
-<segment>
-<pinref part="P+3" gate="1" pin="+12V"/>
-<pinref part="U1" gate="A" pin="4"/>
-<wire x1="241.3" y1="210.82" x2="241.3" y2="208.28" width="0.1524" layer="91"/>
-</segment>
-<segment>
-<pinref part="P+4" gate="1" pin="+12V"/>
-<pinref part="U2" gate="A" pin="4"/>
-<wire x1="241.3" y1="109.22" x2="241.3" y2="106.68" width="0.1524" layer="91"/>
-</segment>
-<segment>
-<pinref part="P+7" gate="1" pin="+12V"/>
-<pinref part="U4" gate="A" pin="4"/>
-<wire x1="424.18" y1="109.22" x2="424.18" y2="106.68" width="0.1524" layer="91"/>
-</segment>
-<segment>
-<pinref part="P+8" gate="1" pin="+12V"/>
-<pinref part="U3" gate="A" pin="4"/>
-<wire x1="426.72" y1="213.36" x2="426.72" y2="210.82" width="0.1524" layer="91"/>
-</segment>
-</net>
 <net name="N$4" class="0">
 <segment>
@@
 <wire x1="63.5" y1="93.98" x2="66.04" y2="93.98" width="0.1524" layer="91"/>
 <label x="50.8" y="99.06" size="1.778" layer="95"/>
-<pinref part="X4" gate="-1" pin="S"/>
-<pinref part="X4" gate="-2" pin="S"/>
+<pinref part="SC+" gate="-1" pin="S"/>
+<pinref part="SC+" gate="-2" pin="S"/>
 </segment>
 </net>
@@
 <wire x1="96.52" y1="93.98" x2="99.06" y2="93.98" width="0.1524" layer="91"/>
 <label x="83.82" y="99.06" size="1.778" layer="95"/>
-<pinref part="X6" gate="-1" pin="S"/>
-<pinref part="X6" gate="-2" pin="S"/>
-</segment>
-<segment>
+<pinref part="SC-" gate="-1" pin="S"/>
+<pinref part="SC-" gate="-2" pin="S"/>
+</segment>
+<segment>

Commit message: PROJ - Final pre-purchase revisions (4 boards still in progress.)
Parts:
- renumbered 12V-ISO to +12V-ISO.1, GND to GND.1, VCC to VCC.1, X2 to INPUT
Changed lines of the file:
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@@
 </classes>
 <parts>
-<part name="12V-ISO" library="con-molex" library_urn="urn:adsk.eagle:library:165" deviceset="5566-2" device="" package3d_urn="urn:adsk.eagle:package:8078583/1"/>
-<part name="VCC" library="con-molex" library_urn="urn:adsk.eagle:library:165" deviceset="5566-2" device="" package3d_urn="urn:adsk.eagle:package:8078583/1"/>
-<part name="GND" library="con-molex" library_urn="urn:adsk.eagle:library:165" deviceset="5566-2" device="" package3d_urn="urn:adsk.eagle:package:8078583/1"/>
+<part name="+12V-ISO.1" library="con-molex" library_urn="urn:adsk.eagle:library:165" deviceset="5566-2" device="" package3d_urn="urn:adsk.eagle:package:8078583/1"/>
+<part name="VCC.1" library="con-molex" library_urn="urn:adsk.eagle:library:165" deviceset="5566-2" device="" package3d_urn="urn:adsk.eagle:package:8078583/1"/>
+<part name="GND.1" library="con-molex" library_urn="urn:adsk.eagle:library:165" deviceset="5566-2" device="" package3d_urn="urn:adsk.eagle:package:8078583/1"/>
 <part name="SC+" library="con-molex" library_urn="urn:adsk.eagle:library:165" deviceset="5566-2" device="" package3d_urn="urn:adsk.eagle:package:8078583/1"/>
 <part name="SC-" library="con-molex" library_urn="urn:adsk.eagle:library:165" deviceset="5566-2" device="" package3d_urn="urn:adsk.eagle:package:8078583/1"/>
@@
 <part name="GND8" library="supply1" library_urn="urn:adsk.eagle:library:371" deviceset="GND" device=""/>
 <part name="U3" library="IowaFormula" deviceset="G5LE-1A-E-DC12" device=""/>
-<part name="X2" library="con-molex" library_urn="urn:adsk.eagle:library:165" deviceset="5566-4" device="" package3d_urn="urn:adsk.eagle:package:8078582/1"/>
+<part name="INPUT" library="con-molex" library_urn="urn:adsk.eagle:library:165" deviceset="5566-4" device="" package3d_urn="urn:adsk.eagle:package:8078582/1"/>
 <part name="NOT1" library="74xx-us" library_urn="urn:adsk.eagle:library:88" deviceset="74*19" device="D" package3d_urn="urn:adsk.eagle:package:2917/1" technology="LS"/>
 <part name="BSPD" library="con-lstb" library_urn="urn:adsk.eagle:library:162" deviceset="MA03-1" device="" package3d_urn="urn:adsk.eagle:package:8339/1"/>
@@
 </plain>
 <instances>
-<instance part="12V-ISO" gate="-1" x="30.48" y="127" smashed="yes">
+<instance part="+12V-ISO.1" gate="-1" x="30.48" y="127" smashed="yes">
 <attribute name="NAME" x="33.02" y="126.238" size="1.524" layer="95"/>
 <attribute name="VALUE" x="29.718" y="128.397" size="1.778" layer="96"/>
 </instance>
-<instance part="12V-ISO" gate="-2" x="30.48" y="121.92" smashed="yes">
+<instance part="+12V-ISO.1" gate="-2" x="30.48" y="121.92" smashed="yes">
 <attribute name="NAME" x="33.02" y="121.158" size="1.524" layer="95"/>
 <attribute name="VALUE" x="29.718" y="123.317" size="1.778" layer="96"/>
 </instance>
-<instance part="VCC" gate="-1" x="68.58" y="127" smashed="yes">
+<instance part="VCC.1" gate="-1" x="68.58" y="127" smashed="yes">
 <attribute name="NAME" x="71.12" y="126.238" size="1.524" layer="95"/>
 <attribute name="VALUE" x="67.818" y="128.397" size="1.778" layer="96"/>
 </instance>
-<instance part="VCC" gate="-2" x="68.58" y="121.92" smashed="yes">
+<instance part="VCC.1" gate="-2" x="68.58" y="121.92" smashed="yes">
 <attribute name="NAME" x="71.12" y="121.158" size="1.524" layer="95"/>
 <attribute name="VALUE" x="67.818" y="123.317" size="1.778" layer="96"/>
 </instance>
-<instance part="GND" gate="-1" x="101.6" y="127" smashed="yes">
+<instance part="GND.1" gate="-1" x="101.6" y="127" smashed="yes">
 <attribute name="NAME" x="104.14" y="126.238" size="1.524" layer="95"/>
 <attribute name="VALUE" x="100.838" y="128.397" size="1.778" layer="96"/>
 </instance>
-<instance part="GND" gate="-2" x="101.6" y="121.92" smashed="yes">
+<instance part="GND.1" gate="-2" x="101.6" y="121.92" smashed="yes">
 <attribute name="NAME" x="104.14" y="121.158" size="1.524" layer="95"/>
 <attribute name="VALUE" x="100.838" y="123.317" size="1.778" layer="96"/>
@@
 <attribute name="VALUE" x="417.6014" y="185.1406" size="2.0828" layer="96" ratio="6" rot="SR90"/>
 </instance>
-<instance part="X2" gate="-1" x="38.1" y="78.74" smashed="yes">
+<instance part="INPUT" gate="-1" x="38.1" y="78.74" smashed="yes">
 <attribute name="NAME" x="40.64" y="77.978" size="1.524" layer="95"/>
 <attribute name="VALUE" x="37.338" y="80.137" size="1.778" layer="96"/>
 </instance>
-<instance part="X2" gate="-2" x="38.1" y="76.2" smashed="yes">
+<instance part="INPUT" gate="-2" x="38.1" y="76.2" smashed="yes">
 <attribute name="NAME" x="40.64" y="75.438" size="1.524" layer="95"/>
 </instance>
-<instance part="X2" gate="-3" x="38.1" y="73.66" smashed="yes">
+<instance part="INPUT" gate="-3" x="38.1" y="73.66" smashed="yes">
 <attribute name="NAME" x="40.64" y="72.898" size="1.524" layer="95"/>
 </instance>
-<instance part="X2" gate="-4" x="38.1" y="71.12" smashed="yes">
+<instance part="INPUT" gate="-4" x="38.1" y="71.12" smashed="yes">
 <attribute name="NAME" x="40.64" y="70.358" size="1.524" layer="95"/>
 </instance>
@@
 <net name="GND" class="0">
 <segment>
-<pinref part="GND" gate="-1" pin="S"/>
+<pinref part="GND.1" gate="-1" pin="S"/>
 <wire x1="99.06" y1="127" x2="96.52" y2="127" width="0.1524" layer="91"/>
 <wire x1="96.52" y1="127" x2="86.36" y2="127" width="0.1524" layer="91"/>
 <wire x1="96.52" y1="127" x2="96.52" y2="121.92" width="0.1524" layer="91"/>
 <junction x="96.52" y="127"/>
-<pinref part="GND" gate="-2" pin="S"/>
+<pinref part="GND.1" gate="-2" pin="S"/>
 <wire x1="96.52" y1="121.92" x2="99.06" y2="121.92" width="0.1524" layer="91"/>
 <label x="86.36" y="127" size="1.778" layer="95"/>
@@
 <wire x1="25.4" y1="121.92" x2="27.94" y2="121.92" width="0.1524" layer="91"/>
 <label x="12.7" y="127" size="1.778" layer="95"/>
-<pinref part="12V-ISO" gate="-1" pin="S"/>
-<pinref part="12V-ISO" gate="-2" pin="S"/>
+<pinref part="+12V-ISO.1" gate="-1" pin="S"/>
+<pinref part="+12V-ISO.1" gate="-2" pin="S"/>
 </segment>
 <segment>
@@
 <wire x1="63.5" y1="121.92" x2="66.04" y2="121.92" width="0.1524" layer="91"/>
 <label x="53.34" y="127" size="1.778" layer="95"/>
-<pinref part="VCC" gate="-1" pin="S"/>
-<pinref part="VCC" gate="-2" pin="S"/>
+<pinref part="VCC.1" gate="-1" pin="S"/>
+<pinref part="VCC.1" gate="-2" pin="S"/>
 </segment>
 <segment>
@@
 <wire x1="10.16" y1="76.2" x2="35.56" y2="76.2" width="0.1524" layer="91"/>
 <label x="10.16" y="76.2" size="1.778" layer="95"/>
-<pinref part="X2" gate="-2" pin="S"/>
+<pinref part="INPUT" gate="-2" pin="S"/>
 </segment>
 <segment>
@@
 <wire x1="35.56" y1="78.74" x2="10.16" y2="78.74" width="0.1524" layer="91"/>
 <label x="10.16" y="78.74" size="1.778" layer="95"/>
-<pinref part="X2" gate="-1" pin="S"/>
+<pinref part="INPUT" gate="-1" pin="S"/>
 </segment>
 <segment>
@@
 <wire x1="10.16" y1="73.66" x2="35.56" y2="73.66" width="0.1524" layer="91"/>
 <label x="10.16" y="73.66" size="1.778" layer="95"/>
-<pinref part="X2" gate="-3" pin="S"/>
+<pinref part="INPUT" gate="-3" pin="S"/>
 </segment>
 <segment>
@@
 <wire x1="10.16" y1="71.12" x2="35.56" y2="71.12" width="0.1524" layer="91"/>
 <label x="10.16" y="71.12" size="1.778" layer="95"/>
-<pinref part="X2" gate="-4" pin="S"/>
-</segment>
-<segment>
+<pinref part="INPUT" gate="-4" pin="S"/>
+</segment>
+<segment>
