File: projects/PCB schematics/SC/SC.sch (EAGLE design)
At the start: 76 parts, among them X1 5566-10, X2 5566-2, X4 5566-12

Commit message: TEMP - Initial board placement.
Connections:
- net AUX1: now also R42.1; no longer BUF2B.I
- net AUX1_LED: now also BUF2B.I
- net AUX1_O: no longer R42.1
- net AUX2: now also R43.1; no longer BUF2C.I
- net AUX2_LED: now also BUF2C.I
- net AUX2_O: no longer R43.1
- net BMSFAULT: now also R33.1; no longer BUF1E.I
- net BMSFAULT_LED: now also BUF1E.I
- net BMSFAULT_O: no longer R33.1
- net BSPDFAULT: now also R19.1; no longer BUF1A.I
- net BSPDFAULT_LED: now also BUF1A.I
- net BSPDFAULT_O: no longer R19.1
- net BSPDPLAUS1: now also R20.1; no longer BUF1B.I
- net BSPDPLAUS1_LED: now also BUF1B.I
- net BSPDPLAUS1_O: no longer R20.1
- net BSPDPLAUS2: now also R21.1; no longer BUF1C.I
- net BSPDPLAUS2_LED: now also BUF1C.I
- net BSPDPLAUS2_O: no longer R21.1
- net FUSEFAULT: now also R41.1; no longer BUF2A.I
- net FUSEFAULT_LED: now also BUF2A.I
- net FUSEFAULT_O: no longer R41.1
- net IMDFAULT: now also R32.1; no longer BUF1D.I
- net IMDFAULT_LED: now also BUF1D.I
- net IMDFAULT_O: no longer R32.1
- net TEMPFAULT: now also R34.1; no longer BUF1F.I
- net TEMPFAULT_LED: now also BUF1F.I
- net TEMPFAULT_O: no longer R34.1

Commit message: TEMP - Initial board placement; Horizontal redo.
Connections:
- new net GND1: AUX1.3, AUX2.3, BMS.3, BSPDPLAUS2.3, FUSE.3, IMD.3, TEMP.3
- new net N$20: BSPD.3
- net AUX1_B: no longer BUF2B.O
- net AUX2_B: no longer BUF2C.O
- net BMSFAULT_B: no longer BUF1E.O
- net BSPDFAULT_B: no longer BUF1A.O
- net BSPDPLAUS1_B: no longer BUF1B.O
- net BSPDPLAUS1_O: no longer BSPDPLAUS1.2
- net BSPDPLAUS2_B: no longer BUF1C.O
- net FUSEFAULT_B: no longer BUF2A.O
- net GND: no longer AUX1.3, AUX2.3, BMS.3, BSPD.3, BSPDPLAUS1.3, BSPDPLAUS2.3, FUSE.3, IMD.3, TEMP.3
- net IMDFAULT_B: no longer BUF1D.O
- net TEMPFAULT_B: no longer BUF1F.O
Other:
- moved on the sheet: AUX1, AUX2, BMS, BSPD, BSPDPLAUS1, BSPDPLAUS2, FUSE, IMD, TEMP

Commit message: SC - Hand routing. Ready for autorouter.
Parts:
- removed BUF5: 74HC7014, IowaFormula:74HC7014
- removed X4: 5566-12, con-molex:5566-12
- added R26, R27, R28, R38, R39, R40: 10k, rcl:R-US_R0805
- added R47, R48, R49: 47k, rcl:R-US_R0805
- added X3: 5566-10, con-molex:5566-10
- BUF4: value 74HC7014 -> 74AUC1G17DBV; device IowaFormula:74HC7014 -> 74xx-little-us:74AUC1G17DBV
- C1, C2, C3, C4, C5, C6, C7, C8, C9: value 1 uF -> 1u
- NOR1, NOR2, NOR3, NOR4, NOR5: value 74LS02D -> 74ALS02D; device 74xx-us:74LS02D -> 74xx-us:74ALS02D
- R1, R13, R14, R15, R2, R3, R44, R45, R46, R7, R8, R9: value 10k -> 47k
- R18, R19, R20, R21, R32, R33, R34: value 50k -> 10k
- R36: value 10k -> 50k
- R41, R42, R43: value 50k -> 47k
- X1: value 5566-10 -> 5566-2; device con-molex:5566-10 -> con-molex:5566-2
- X2: value 5566-2 -> 5566-12; device con-molex:5566-2 -> con-molex:5566-12
Connections:
- removed net AUX1_O: AUX1.2, OR2C.I1, R8.2
- removed net AUX2_O: AUX2.2, OR2D.I1, R9.2
- removed net BMSFAULT_O: BMS.2, OR1D.I1, R5.2
- removed net BSPDFAULT_O: BSPD.2, OR1A.I0, R2.2
- removed net BSPDPLAUS1_O: OR1A.I1, R1.2
- removed net BSPDPLAUS2_O: BSPDPLAUS2.2, OR1B.I1, R3.2
- removed net FUSEFAULT_O: FUSE.2, OR2B.I1, R7.2
- removed net GND1: AUX1.3, AUX2.3, BMS.3, BSPDPLAUS2.3, FUSE.3, IMD.3, TEMP.3
- removed net IMDFAULT_O: IMD.2, OR1C.I1, R4.2
- removed net N$20: BSPD.3
- removed net TEMPFAULT_O: OR2A.I1, R6.2, TEMP.2
- net AIR_CONTROL: now also X3-10.S; no longer X1-10.S
- net AUX1: now also R14.1, R48.1, X2-8.S; no longer R42.1, X4-8.S
- net AUX1_B: now also BUF2B.O
- net AUX1_LED: now also BUF3E.O, OR2C.I1, R26.2, X3-8.S; no longer BUF2B.I, BUF4A.O, X1-8.S
- net AUX2: now also R15.1, R49.1, X2-9.S; no longer R43.1, X4-9.S
- net AUX2_B: now also BUF2C.O
- net AUX2_LED: now also BUF3F.O, OR2D.I1, R27.2, X3-9.S; no longer BUF2C.I, BUF4C.O, X1-9.S
- net BMSFAULT: now also R45.1, R8.1, X2-5.S; no longer R33.1, X4-5.S
- net BMSFAULT_B: now also BUF1E.O
- net BMSFAULT_LED: now also BUF3B.O, OR1D.I1, R23.2, X3-5.S; no longer BUF1E.I, BUF5A.O, X1-5.S
- net BSPDFAULT: now also R1.1, R41.1, X2-1.S; no longer R19.1, X4-1.S
- net BSPDFAULT_B: now also BUF1A.O
- net BSPDFAULT_LED: now also BUF2D.O, OR1A.I0, R20.2, X3-1.S; no longer BUF1A.I, BUF2E.O, X1-1.S
- net BSPDPLAUS1: now also R2.1, R42.1, X2-2.S; no longer R20.1, X4-2.S
- net BSPDPLAUS1_B: now also BUF1B.O
- net BSPDPLAUS1_LED: now also BUF2E.O, OR1A.I1, R19.2, X3-2.S; no longer BUF1B.I, BUF3A.O, X1-2.S
- net BSPDPLAUS2: now also R3.1, R43.1, X2-3.S; no longer R21.1, X4-3.S
- net BSPDPLAUS2_B: now also BUF1C.O
- net BSPDPLAUS2_LED: now also BUF2F.O, OR1B.I1, R21.2, X3-3.S; no longer BUF1C.I, BUF3C.O, X1-3.S
- net FUSEFAULT: now also R13.1, R47.1, X2-7.S; no longer R41.1, X4-7.S
- net FUSEFAULT_B: now also BUF2A.O
- net FUSEFAULT_LED: now also BUF3D.O, OR2B.I1, R25.2, X3-7.S; no longer BUF2A.I, BUF5E.O, X1-7.S
- net GND: now also AUX1.3, AUX2.3, BMS.3, BSPD.3, BSPDPLAUS1.3, BSPDPLAUS2.3, FUSE.3, IMD.3, R18.1, R19.1, R20.1, R21.1, R26.1, R27.1, R28.1, R32.1, R33.1, R34.1, R38.1, R39.1, R40.1, TEMP.3, X1-2.S; no longer R1.1, R13.1, R14.1, R15.1, R2.1, R3.1, R36.1, R44.1, R45.1, R46.1, R7.1, R8.1, R9.1, X2-2.S
- net IMDFAULT: now also R44.1, R7.1, X2-4.S; no longer R32.1, X4-4.S
- net IMDFAULT_B: now also BUF1D.O
- net IMDFAULT_LED: now also BUF3A.O, OR1C.I1, R22.2, X3-4.S; no longer BUF1D.I, BUF3E.O, X1-4.S
- net N$1: now also R33.2; no longer R15.2
- net N$10: now also BUF1F.I, C6.1, R9.2; no longer BUF5B.I, C7.1, R34.2
- net N$11: now also R35.2, R36.1; no longer R17.2, R18.1
- net N$12: now also R29.2; no longer R11.2
- net N$13: now also R30.2; no longer R12.2
- net N$14: now also R31.2; no longer R13.2
- net N$15: now also BUF2A.I, C7.1, R13.2; no longer BUF5D.I, C8.1, R41.2
- net N$16: now also BUF2B.I, C8.1, R14.2; no longer BUF5F.I, C9.1, R42.2
- net N$17: now also R32.2; no longer R14.2
- net N$18: now also BUF1A.I, C1.1, R1.2; no longer BUF2D.I, C2.1, R19.2
- net N$19: now also BUF2C.I, C9.1, R15.2; no longer BUF4B.I, C10.1, R43.2
- net N$2: now also R34.2; no longer R16.2
- net N$3: now also R28.2; no longer R10.2
- net N$4: now also BUF1B.I, C2.1, R2.2; no longer BUF2F.I, C3.1, R20.2
- net N$5: now also BUF1C.I, C3.1, R3.2; no longer BUF3B.I, C4.1, R21.2
- net N$6: now also BUF4G$1.I, C10.1, R36.2; no longer BUF4D.I, C1.1, R18.2
- net N$7: now also BUF1D.I, C4.1, R7.2; no longer BUF3D.I, C5.1, R32.2
- net N$8: now also R39.2; no longer R30.2
- net N$9: now also BUF1E.I, C5.1, R8.2; no longer BUF3F.I, C6.1, R33.2
- net Q: now also NOR5C.I1, NOR5D.O; no longer NOR1A.I1, NOR1B.O
- net Q_AUX1: now also BUF3E.I, NOR4C.I1, NOR4D.O; no longer BUF4A.I, NOR5A.I1, NOR5B.O
- net Q_AUX2: now also BUF3F.I, NOR5A.I1, NOR5B.O; no longer BUF4C.I, NOR5C.I1, NOR5D.O
- net Q_BMSFAULT: now also BUF3B.I, NOR3A.I1, NOR3B.O; no longer BUF5A.I, NOR3C.I1, NOR3D.O
- net Q_BSPDFAULT: now also BUF2D.I, NOR1A.I1, NOR1B.O; no longer BUF2E.I, NOR1C.I1, NOR1D.O
- net Q_BSPDPLAUS1: now also BUF2E.I, NOR1C.I1, NOR1D.O; no longer BUF3A.I, NOR2A.I1, NOR2B.O
- net Q_BSPDPLAUS2: now also BUF2F.I, NOR2A.I1, NOR2B.O; no longer BUF3C.I, NOR2C.I1, NOR2D.O
- net Q_FUSEFAULT: now also BUF3D.I, NOR4A.I1, NOR4B.O; no longer BUF5E.I, NOR4C.I1, NOR4D.O
- net Q_IMDFAULT: now also BUF3A.I, NOR2C.I1, NOR2D.O; no longer BUF3E.I, NOR3A.I1, NOR3B.O
- net Q_TEMPFAULT: now also BUF3C.I, NOR3C.I1, NOR3D.O; no longer BUF5C.I, NOR4A.I1, NOR4B.O
- net RESET_MAINFAULT: now also R38.2, X2-11.S; no longer R29.2, X4-11.S
- net SCU_CONTROL: now also R40.2, X2-10.S; no longer R31.2, X4-10.S
- net SET_AUX1: now also AUX1.2, NOR4C.I0, R17.2; no longer BUF5F.O, NOR5A.I0, R45.2
- net SET_AUX2: now also AUX2.2, NOR5A.I0, R18.2; no longer BUF4B.O, NOR5C.I0, R46.2
- net SET_BMSFAULT: now also BMS.2, NOR3A.I0, R11.2; no longer BUF3F.O, NOR3C.I0, R36.2
- net SET_BSPDFAULT: now also BSPD.2, NOR1A.I0, R4.2; no longer BUF2D.O, NOR1C.I0, R22.2
- net SET_BSPDPLAUS1: now also BSPDPLAUS1.2, NOR1C.I0, R5.2; no longer BUF2F.O, NOR2A.I0, R23.2
- net SET_BSPDPLAUS2: now also BSPDPLAUS2.2, NOR2A.I0, R6.2; no longer BUF3B.O, NOR2C.I0, R24.2
- net SET_FUSEFAULT: now also FUSE.2, NOR4A.I0, R16.2; no longer BUF5D.O, NOR4C.I0, R44.2
- net SET_IMDFAULT: now also IMD.2, NOR2C.I0, R10.2; no longer BUF3D.O, NOR3A.I0, R35.2
- net SET_MAINFAULT: now also BUF4G$1.O, NOR5C.I0, R37.2; no longer BUF4D.O, NOR1A.I0, R25.2
- net SET_TEMPFAULT: now also NOR3C.I0, R12.2, TEMP.2; no longer BUF5B.O, NOR4A.I0, R37.2
- net TEMPFAULT: now also R46.1, R9.1, X2-6.S; no longer R34.1, X4-6.S
- net TEMPFAULT_B: now also BUF1F.O
- net TEMPFAULT_LED: now also BUF3C.O, OR2A.I1, R24.2, X3-6.S; no longer BUF1F.I, BUF5C.O, X1-6.S
- net VCC: now also R41.2, R42.2, R43.2, R44.2, R45.2, R46.2, R47.2, R48.2, R49.2, X1-1.S; no longer X2-1.S
- net ~Q: now also NOR5C.O, NOR5D.I0; no longer NOR1A.O, NOR1B.I0
- net ~Q_AUX1: now also NOR4C.O, NOR4D.I0; no longer NOR5A.O, NOR5B.I0
- net ~Q_AUX2: now also NOR5A.O, NOR5B.I0; no longer NOR5C.O, NOR5D.I0
- net ~Q_BMSFAULT: now also NOR3A.O, NOR3B.I0; no longer NOR3C.O, NOR3D.I0
- net ~Q_BSPDFAULT: now also NOR1A.O, NOR1B.I0; no longer NOR1C.O, NOR1D.I0
- net ~Q_BSPDPLAUS1: now also NOR1C.O, NOR1D.I0; no longer NOR2A.O, NOR2B.I0
- net ~Q_BSPDPLAUS2: now also NOR2A.O, NOR2B.I0; no longer NOR2C.O, NOR2D.I0
- net ~Q_FUSEFAULT: now also NOR4A.O, NOR4B.I0; no longer NOR4C.O, NOR4D.I0
- net ~Q_IMDFAULT: now also NOR2C.O, NOR2D.I0; no longer NOR3A.O, NOR3B.I0
- net ~Q_TEMPFAULT: now also NOR3C.O, NOR3D.I0; no longer NOR4A.O, NOR4B.I0
Other:
- note added: "Note: Associated pull-down resistor for AIR_CONTROL is on CHARGE"
- moved on the sheet: AND1, AUX1, AUX2, BMS, BSPD, BSPDPLAUS1, BSPDPLAUS2, BUF1A, BUF1B, BUF1C, BUF1D, BUF1E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

Commit message: SC - Stage initial placement.
Parts:
- removed AUX2: (no value), con-lstb:MA03-1
- removed C9: 1u, rcl:C-USC0805
- removed R15, R49: 47k, rcl:R-US_R0805
- removed R18, R27: 10k, rcl:R-US_R0805
Connections:
- removed net AUX2_B: AUX2.1, BUF2C.O
- removed net AUX2_LED: BUF3F.O, OR2D.I1, R27.2, X3-9.S
- removed net N$11: OR2D.O, R35.2, R36.1
- removed net N$19: BUF2C.I, C9.1, R15.2
- removed net Q_AUX2: BUF3F.I, NOR5A.I1, NOR5B.O
- removed net SET_AUX2: AUX2.2, NOR5A.I0, R18.2
- removed net ~Q_AUX2: NOR5A.O, NOR5B.I0
- net AUX2: no longer R15.1, R49.1
- net GND: no longer AUX2.3, C9.2, R18.1, R27.1
- net N$2: now also R35.2, R36.1; no longer OR2D.I0
- net RESET_MAINFAULT: no longer NOR5B.I1
- net VCC: no longer R49.2
Other:
- moved on the sheet: OR1A, OR1B, OR1C, OR1D, OR2A, OR2B, OR2C

Commit message: PROJ - Final pre-purchase revisions (4 boards still in progress.)
Parts:
- renumbered X2 to INPUT, X3 to OUTPUT

Commit message: PROJ - Gerber files major milestone - 05/05/19.
Connections:
- removed net AUX2: INPUT-9.S
Changed lines of the file:
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@@
-</segment>
-</net>
-<net name="AUX2" class="0">
-<segment>
-<wire x1="2.54" y1="86.36" x2="22.86" y2="86.36" width="0.1524" layer="91"/>
-<label x="0" y="86.36" size="1.778" layer="95"/>
-<pinref part="INPUT" gate="-9" pin="S"/>
 </segment>
 </net>
@@
 <wire x1="698.5" y1="269.24" x2="721.36" y2="269.24" width="0.1524" layer="91"/>
 <label x="698.5" y="269.24" size="1.778" layer="95"/>
+<junction x="721.36" y="269.24"/>
 </segment>
 </net>
@@
 <wire x1="701.04" y1="233.68" x2="721.36" y2="233.68" width="0.1524" layer="91"/>
 <label x="701.04" y="233.68" size="1.778" layer="95"/>
+<junction x="721.36" y="233.68"/>
 </segment>
 </net>
@@
 <wire x1="701.04" y1="203.2" x2="721.36" y2="203.2" width="0.1524" layer="91"/>
 <label x="701.04" y="203.2" size="1.778" layer="95"/>
+<junction x="721.36" y="203.2"/>
 </segment>
 </net>
@@
 <wire x1="701.04" y1="144.78" x2="721.36" y2="144.78" width="0.1524" layer="91"/>
 <label x="701.04" y="144.78" size="1.778" layer="95"/>
+<junction x="721.36" y="144.78"/>
 </segment>
 </net>
@@
 <wire x1="701.04" y1="119.38" x2="721.36" y2="119.38" width="0.1524" layer="91"/>
 <label x="701.04" y="119.38" size="1.778" layer="95"/>
+<junction x="721.36" y="119.38"/>
 </segment>
 </net>
@@
 <wire x1="721.36" y1="86.36" x2="701.04" y2="86.36" width="0.1524" layer="91"/>
 <label x="701.04" y="86.36" size="1.778" layer="95"/>
+<junction x="721.36" y="86.36"/>
 </segment>
 </net>
@@
 <wire x1="701.04" y1="172.72" x2="721.36" y2="172.72" width="0.1524" layer="91"/>
 <label x="701.04" y="172.72" size="1.778" layer="95"/>
-</segment>
-</net>
+<junction x="721.36" y="172.72"/>
+</segment>
+</net>
