File: projects/PCB schematics/TEMP/TEMP.brd (EAGLE design)
At the start: 73.7 x 83.8 mm, 58 parts, among them J1 770968-1, J2 770968-1, J3 1-770969-0, J4 770966-1

Commit message: PROJ - Final pre-purchase revisions (4 boards still in progress.)
Parts:
- removed J1, J2: 770968-1, IowaFormula:CONN4_770968-1
- removed J3: 1-770969-0, IowaFormula:CON6_2X3_P163_RAMNL
- removed J4: 770966-1, IowaFormula:CONN2_770966-1
- added CS.1, CS.2: 770968-1, IowaFormula:CONN4_770968-1
- added TEMP_OUT: 1-770969-0, IowaFormula:CON6_2X3_P163_RAMNL
- added VCC/GND: 770966-1, IowaFormula:CONN2_770966-1
- moved R17 4.58 mm to (67.8, 51.1)
- moved R18 4.58 mm to (67.8, 53.2)
- moved R20 4.58 mm to (67.8, 49.1)
- moved R22 4.58 mm to (52.2, 49.0)
- moved R44 4.58 mm to (66.2, 42.1)
- moved MUX4 4.58 mm to (21.6, 35.6)
- moved MUX5 4.58 mm to (40.6, 35.6)
- moved R1 4.58 mm to (29.9, 51.2)
- moved R12 4.58 mm to (48.2, 49.0)
- moved R2 4.58 mm to (29.9, 53.2)
- moved R26 4.58 mm to (29.8, 38.1)
- moved R27 4.58 mm to (29.9, 40.2)
- moved R29 4.58 mm to (14.2, 40.2)
- moved R3 4.58 mm to (29.9, 55.3)
- moved R31 4.58 mm to (14.2, 38.1)
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Connections:
- net CS_A_IN: now also CS.1.1; no longer J1.1
- net CS_A_OUT: now also CS.2.1; no longer J2.1
- net CS_B_IN: now also CS.1.2; no longer J1.2
- net CS_B_OUT: now also CS.2.2; no longer J2.2
- net CS_C_IN: now also CS.1.3; no longer J1.3
- net CS_C_OUT: now also CS.2.3; no longer J2.3
- net GND: now also VCC/GND.2; no longer J4.2
- net TEMP_OUT1: now also TEMP_OUT.1; no longer J3.1
- net TEMP_OUT2: now also TEMP_OUT.2; no longer J3.2
- net TEMP_OUT3: now also TEMP_OUT.3; no longer J3.3
- net TEMP_OUT4: now also TEMP_OUT.4; no longer J3.4
- net TEMP_OUT5: now also TEMP_OUT.5; no longer J3.5
- net VCC: now also VCC/GND.1; no longer J4.1
Routing:
- net TEMP29: track 72.9 -> 73.5 mm
- net TEMP30: track 51.6 -> 52.2 mm
Other:
- board size 73.7 x 83.8 mm -> 78.7 x 83.8 mm
- board text added: "1."
- board text added: "CS.1: 1. CS_A_IN 2. CS_B_IN 3. CS_C_IN"
- board text added: "CS.2: 1. CS_A_OUT 2. CS_B_OUT 3. CS_C_OUT"
- board text added: "VCC/GND: 1. VCC 2. GND"

Commit message: PROJ - Gerber files major milestone - 05/05/19.
Routing:
- net TEMP23: track 115.0 -> 116.7 mm
- net TEMP21: track 76.7 -> 77.5 mm
- net TEMP_OUT5: track 56.9 -> 57.4 mm
Other:
- board text added: "Temperature Multiplexer (TEMP) Rev. A, May 5th, 2019"
- board text removed: "Temperature Multiplexer (TEMP) Rev. A, April 30th, 2019"
Changed lines of the file:
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@@
 <wire x1="35.687" y1="26.9748" x2="35.687" y2="22.7838" width="0.1524" layer="25"/>
 <text x="9.5504" y="27.1018" size="1.778" layer="25" font="vector" rot="R90">Temperature Multiplexer (TEMP)
-Rev. A, April 30th, 2019</text>
+Rev. A, May 5th, 2019</text>
 <text x="73.0504" y="35.9918" size="0.8128" layer="25" font="vector" rot="R90">Author: github.com/michaelpass</text>
 <text x="69.85" y="67.31" size="1.016" layer="25">VCC/GND:
@@
 <wire x1="17.78" y1="37.5412" x2="18.3896" y2="37.5412" width="0.2032" layer="1"/>
 <wire x1="16.5608" y1="38.7604" x2="17.78" y2="37.5412" width="0.2032" layer="1"/>
-<wire x1="16.5608" y1="42.6212" x2="16.5608" y2="38.7604" width="0.2032" layer="1"/>
-<wire x1="11.0744" y1="48.1076" x2="16.5608" y2="42.6212" width="0.2032" layer="1"/>
-<wire x1="11.0744" y1="63.754" x2="11.0744" y2="48.1076" width="0.2032" layer="1"/>
-<wire x1="13.3096" y1="65.9892" x2="11.0744" y2="63.754" width="0.2032" layer="1"/>
+<wire x1="16.5608" y1="41.9354" x2="16.5608" y2="38.7604" width="0.2032" layer="1"/>
+<wire x1="10.5156" y1="47.9806" x2="16.5608" y2="41.9354" width="0.2032" layer="1"/>
+<wire x1="10.5156" y1="63.1952" x2="10.5156" y2="47.9806" width="0.2032" layer="1"/>
+<wire x1="13.3096" y1="65.9892" x2="10.5156" y2="63.1952" width="0.2032" layer="1"/>
 <wire x1="18.3896" y1="37.5412" x2="18.5166" y2="37.465" width="0.2032" layer="1"/>
 <wire x1="13.3096" y1="65.9892" x2="13.3096" y2="66.04" width="0.2032" layer="1"/>
@@
 <wire x1="35.052" y1="45.2628" x2="38.9128" y2="41.402" width="0.2032" layer="1"/>
 <wire x1="28.5496" y1="45.2628" x2="35.052" y2="45.2628" width="0.2032" layer="16"/>
-<wire x1="14.5288" y1="45.2628" x2="28.5496" y2="45.2628" width="0.2032" layer="1"/>
-<wire x1="11.4808" y1="48.3108" x2="14.5288" y2="45.2628" width="0.2032" layer="1"/>
-<wire x1="11.4808" y1="62.738" x2="11.4808" y2="48.3108" width="0.2032" layer="1"/>
-<wire x1="13.3096" y1="64.5668" x2="11.4808" y2="62.738" width="0.2032" layer="1"/>
-<wire x1="15.9512" y1="64.5668" x2="13.3096" y2="64.5668" width="0.2032" layer="1"/>
-<wire x1="17.3736" y1="65.9892" x2="15.9512" y2="64.5668" width="0.2032" layer="1"/>
+<wire x1="14.2494" y1="45.2628" x2="28.5496" y2="45.2628" width="0.2032" layer="1"/>
+<wire x1="11.2268" y1="48.2854" x2="14.2494" y2="45.2628" width="0.2032" layer="1"/>
+<wire x1="11.2268" y1="62.738" x2="11.2268" y2="48.2854" width="0.2032" layer="1"/>
+<wire x1="12.827" y1="64.3382" x2="11.2268" y2="62.738" width="0.2032" layer="1"/>
+<wire x1="15.7226" y1="64.3382" x2="12.827" y2="64.3382" width="0.2032" layer="1"/>
+<wire x1="17.3736" y1="65.9892" x2="15.7226" y2="64.3382" width="0.2032" layer="1"/>
 <wire x1="37.6936" y1="37.5412" x2="37.5666" y2="37.465" width="0.2032" layer="1"/>
 <wire x1="17.3736" y1="65.9892" x2="17.4498" y2="66.04" width="0.2032" layer="1"/>
@@
 <wire x1="14.732" y1="60.2996" x2="14.732" y2="65.786" width="0.2032" layer="16"/>
 <wire x1="12.9032" y1="58.4708" x2="14.732" y2="60.2996" width="0.2032" layer="16"/>
-<wire x1="12.0904" y1="57.658" x2="12.9032" y2="58.4708" width="0.2032" layer="1"/>
-<wire x1="12.0904" y1="48.3108" x2="12.0904" y2="57.658" width="0.2032" layer="1"/>
-<wire x1="14.732" y1="45.6692" x2="12.0904" y2="48.3108" width="0.2032" layer="1"/>
+<wire x1="11.9888" y1="57.5564" x2="12.9032" y2="58.4708" width="0.2032" layer="1"/>
+<wire x1="11.9888" y1="48.4124" x2="11.9888" y2="57.5564" width="0.2032" layer="1"/>
+<wire x1="14.732" y1="45.6692" x2="11.9888" y2="48.4124" width="0.2032" layer="1"/>
 <wire x1="21.0312" y1="45.6692" x2="14.732" y2="45.6692" width="0.2032" layer="1"/>
 <wire x1="22.86" y1="47.498" x2="21.0312" y2="45.6692" width="0.2032" layer="1"/>
@@
 <contactref element="R36" pad="2"/>
 <contactref element="TEMP21-40" pad="31"/>
-<wire x1="49.0728" y1="32.0548" x2="48.4632" y2="32.6644" width="0.2032" layer="1"/>
+<wire x1="48.6664" y1="32.4612" x2="48.4632" y2="32.6644" width="0.2032" layer="1"/>
 <wire x1="48.4632" y1="32.6644" x2="47.244" y2="33.8836" width="0.2032" layer="1"/>
-<wire x1="55.5752" y1="32.0548" x2="49.0728" y2="32.0548" width="0.2032" layer="1"/>
-<wire x1="58.2168" y1="29.4132" x2="55.5752" y2="32.0548" width="0.2032" layer="1"/>
-<wire x1="58.2168" y1="12.7508" x2="58.2168" y2="29.4132" width="0.2032" layer="1"/>
+<wire x1="55.6768" y1="32.4612" x2="48.6664" y2="32.4612" width="0.2032" layer="1"/>
+<wire x1="58.2168" y1="29.9212" x2="55.6768" y2="32.4612" width="0.2032" layer="1"/>
+<wire x1="58.2168" y1="12.7508" x2="58.2168" y2="29.9212" width="0.2032" layer="1"/>
 <wire x1="54.5592" y1="9.0932" x2="58.2168" y2="12.7508" width="0.2032" layer="1"/>
 <wire x1="49.276" y1="9.0932" x2="54.5592" y2="9.0932" width="0.2032" layer="1"/>
@@
 <wire x1="54.9656" y1="79.1972" x2="55.5752" y2="79.1972" width="0.2032" layer="1"/>
 <wire x1="54.5592" y1="79.6036" x2="54.9656" y2="79.1972" width="0.2032" layer="1"/>
-<wire x1="28.5496" y1="79.6036" x2="54.5592" y2="79.6036" width="0.2032" layer="1"/>
-<wire x1="15.5448" y1="66.5988" x2="28.5496" y2="79.6036" width="0.2032" layer="1"/>
-<wire x1="15.5448" y1="65.3796" x2="15.5448" y2="66.5988" width="0.2032" layer="1"/>
+<wire x1="28.1178" y1="79.6036" x2="54.5592" y2="79.6036" width="0.2032" layer="1"/>
+<wire x1="15.5448" y1="67.0306" x2="28.1178" y2="79.6036" width="0.2032" layer="1"/>
+<wire x1="15.5448" y1="65.3796" x2="15.5448" y2="67.0306" width="0.2032" layer="1"/>
 <wire x1="15.5448" y1="56.8452" x2="15.5448" y2="65.3796" width="0.2032" layer="16"/>
 <wire x1="47.4472" y1="73.1012" x2="47.625" y2="72.962" width="0.2032" layer="16"/>
@@
 <wire x1="42.7736" y1="75.3364" x2="45.0088" y2="73.1012" width="0.2032" layer="16"/>
 <wire x1="38.1" y1="75.3364" x2="42.7736" y2="75.3364" width="0.2032" layer="16"/>
-<wire x1="34.6456" y1="78.7908" x2="38.1" y2="75.3364" width="0.2032" layer="1"/>
-<wire x1="28.3464" y1="78.7908" x2="34.6456" y2="78.7908" width="0.2032" layer="1"/>
-<wire x1="18.9992" y1="69.4436" x2="28.3464" y2="78.7908" width="0.2032" layer="1"/>
-<wire x1="18.9992" y1="65.5828" x2="18.9992" y2="69.4436" width="0.2032" layer="1"/>
+<wire x1="34.4678" y1="78.9686" x2="38.1" y2="75.3364" width="0.2032" layer="1"/>
+<wire x1="28.2956" y1="78.9686" x2="34.4678" y2="78.9686" width="0.2032" layer="1"/>
+<wire x1="18.9992" y1="69.6722" x2="28.2956" y2="78.9686" width="0.2032" layer="1"/>
+<wire x1="18.9992" y1="65.5828" x2="18.9992" y2="69.6722" width="0.2032" layer="1"/>
 <wire x1="16.764" y1="63.3476" x2="18.9992" y2="65.5828" width="0.2032" layer="1"/>
 <wire x1="12.7" y1="63.3476" x2="16.764" y2="63.3476" width="0.2032" layer="1"/>
@@
 <wire x1="53.34" y1="55.2196" x2="53.147" y2="55.245" width="0.2032" layer="1"/>
 <wire x1="56.5912" y1="55.2196" x2="56.6166" y2="55.245" width="0.2032" layer="1"/>
-<wire x1="27.7368" y1="11.7348" x2="28.5496" y2="10.922" width="0.2032" layer="1"/>
-<wire x1="27.7368" y1="12.5476" x2="27.7368" y2="11.7348" width="0.2032" layer="1"/>
-<wire x1="33.8328" y1="18.6436" x2="27.7368" y2="12.5476" width="0.2032" layer="1"/>
-<wire x1="56.5912" y1="18.6436" x2="33.8328" y2="18.6436" width="0.2032" layer="1"/>
+<wire x1="28.575" y1="10.858" x2="28.4358" y2="10.858" width="0.2032" layer="1"/>
+<wire x1="28.4358" y1="10.858" x2="27.5336" y2="11.7602" width="0.2032" layer="1"/>
+<wire x1="27.5336" y1="13.3604" x2="27.5336" y2="11.7602" width="0.2032" layer="1"/>
+<wire x1="32.258" y1="18.0848" x2="27.5336" y2="13.3604" width="0.2032" layer="1"/>
+<wire x1="56.5912" y1="18.6436" x2="56.0324" y2="18.0848" width="0.2032" layer="1"/>
+<wire x1="56.0324" y1="18.0848" x2="32.258" y2="18.0848" width="0.2032" layer="1"/>
 <wire x1="59.436" y1="21.4884" x2="56.5912" y2="18.6436" width="0.2032" layer="16"/>
 <wire x1="59.436" y1="39.5732" x2="59.436" y2="21.4884" width="0.2032" layer="1"/>
@@
 <wire x1="57.2008" y1="55.2196" x2="60.0456" y2="52.3748" width="0.2032" layer="1"/>
 <wire x1="56.7944" y1="55.2196" x2="57.2008" y2="55.2196" width="0.2032" layer="1"/>
-<wire x1="28.5496" y1="10.922" x2="28.575" y2="10.858" width="0.2032" layer="1"/>
 <wire x1="56.7944" y1="55.2196" x2="56.6166" y2="55.245" width="0.2032" layer="1"/>
 <via x="56.5912" y="18.6436" extent="1-16" drill="0.508"/>
@@
 <wire x1="24.0792" y1="10.1092" x2="24.0792" y2="11.938" width="0.2032" layer="16"/>
 <wire x1="29.972" y1="4.2164" x2="24.0792" y2="10.1092" width="0.2032" layer="16"/>
-<wire x1="60.0456" y1="4.2164" x2="29.972" y2="4.2164" width="0.2032" layer="16"/>
-<wire x1="68.58" y1="12.7508" x2="60.0456" y2="4.2164" width="0.2032" layer="16"/>
-<wire x1="68.58" y1="45.6692" x2="68.58" y2="12.7508" width="0.2032" layer="16"/>
-<wire x1="60.6552" y1="53.594" x2="68.58" y2="45.6692" width="0.2032" layer="16"/>
+<wire x1="62.5348" y1="4.2164" x2="29.972" y2="4.2164" width="0.2032" layer="16"/>
+<wire x1="68.9356" y1="10.6172" x2="62.5348" y2="4.2164" width="0.2032" layer="16"/>
+<wire x1="68.9356" y1="45.3136" x2="68.9356" y2="10.6172" width="0.2032" layer="16"/>
+<wire x1="60.6552" y1="53.594" x2="68.9356" y2="45.3136" width="0.2032" layer="16"/>
 <wire x1="55.1688" y1="53.594" x2="60.6552" y2="53.594" width="0.2032" layer="16"/>
 <wire x1="54.7624" y1="53.1876" x2="55.1688" y2="53.594" width="0.2032" layer="16"/>
