File: projects/PCB schematics/TSALC/TSAL-GLV.sch (EAGLE design)
At the start: 22 parts, among them Q1 IRLZ44Z, Q2 IRLZ44Z, Q3 IRLZ44Z

Commit message: PROJ - Gerber files major milestone - 05/05/19.
Connections:
- net GND: now also BUF1G$2.GND, NOT1P.GND
- net VCC: now also BUF1G$2.VCC, NOT1P.VCC
Changed lines of the file:
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@@
 <attribute name="VALUE" x="101.6" y="15.24" size="1.778" layer="96"/>
+</instance>
+<instance part="BUF1" gate="G$2" x="119.38" y="35.56" smashed="yes">
+<attribute name="NAME" x="118.745" y="34.925" size="1.778" layer="95"/>
+</instance>
+<instance part="NOT1" gate="P" x="177.8" y="35.56" smashed="yes">
+<attribute name="NAME" x="177.165" y="34.925" size="1.778" layer="95"/>
 </instance>
 </instances>
@@
 <wire x1="104.14" y1="22.86" x2="104.14" y2="20.32" width="0.1524" layer="91"/>
 </segment>
+<segment>
+<pinref part="BUF1" gate="G$2" pin="GND"/>
+<wire x1="119.38" y1="27.94" x2="119.38" y2="22.86" width="0.1524" layer="91"/>
+<wire x1="119.38" y1="22.86" x2="121.92" y2="22.86" width="0.1524" layer="91"/>
+<label x="121.92" y="22.86" size="1.778" layer="95"/>
+</segment>
+<segment>
+<pinref part="NOT1" gate="P" pin="GND"/>
+<wire x1="177.8" y1="27.94" x2="170.18" y2="27.94" width="0.1524" layer="91"/>
+<label x="170.18" y="27.94" size="1.778" layer="95"/>
+</segment>
 </net>
 <net name="+12V-ISO" class="0">
@@
 <label x="276.86" y="104.14" size="1.778" layer="95" rot="R180" xref="yes"/>
 <wire x1="276.86" y1="104.14" x2="279.4" y2="104.14" width="0.1524" layer="91"/>
+<junction x="279.4" y="104.14"/>
 </segment>
 <segment>
@@
 <wire x1="279.4" y1="55.88" x2="276.86" y2="55.88" width="0.1524" layer="91"/>
 <pinref part="SH2" gate="G$1" pin="P$1"/>
+<junction x="279.4" y="55.88"/>
 </segment>
 <segment>
@@
 <label x="10.16" y="86.36" size="1.778" layer="95"/>
 </segment>
+<segment>
+<pinref part="BUF1" gate="G$2" pin="VCC"/>
+<wire x1="119.38" y1="43.18" x2="119.38" y2="45.72" width="0.1524" layer="91"/>
+<wire x1="119.38" y1="45.72" x2="114.3" y2="45.72" width="0.1524" layer="91"/>
+<label x="114.3" y="45.72" size="1.778" layer="95"/>
+</segment>
+<segment>
+<pinref part="NOT1" gate="P" pin="VCC"/>
+<wire x1="177.8" y1="43.18" x2="172.72" y2="43.18" width="0.1524" layer="91"/>
+<label x="172.72" y="43.18" size="1.778" layer="95"/>
+</segment>
 </net>
 <net name="TSAL_CONTROL_SIGNAL" class="0">
@@
 </sheet>
 </sheets>
+<errors>
+</errors>
 </schematic>
 </drawing>
